File: eOPRA_interface/eOPRA_interface.kicad_sch (KiCad schematic)
At the start: 23 parts, among them J1 CONN_01X02_MALE, J2 CONN_01X04_MALE, J3 CONN_01X04_MALE, J4 CONN_01X02_MALE, J5 CONN_01X03_MALE, J7 header_01x02, J8 CONN_01X04_MALE, Q4 Q_PMOS_DGS, U1 ARM-SWD-10, U10 USB_C_2.0, U27 Mounting-holes, U28 Mounting-holes, U5 XT-X, U7 Mounting-holes, U8 Mounting-holes

Commit message: schematic v1.0 finished
Parts:
- removed F3: Fuse, symbol 4.power.circuitProtection:Fuse
- removed J1: CONN_01X02_MALE, symbol 5.connector.interconnect:CONN_01X02_MALE
- removed J5: CONN_01X03_MALE, symbol 5.connector.interconnect:CONN_01X03_MALE
- removed J7: header_01x02, symbol 5.connector.interconnect:header_01x02
- removed Q4: Q_PMOS_DGS, symbol 1.semi.discrete:Q_PMOS_DGS
- removed R11, R12, R18, R19: R, symbol 2.passive:R
- added F1: Fuse, project_footprints:PTC, symbol 4.power.circuitProtection:Fuse
- added J1, J5: CONN_01X04_MALE, project_footprints:JST_SM04B-GHS-TB(LF)(SN)-, symbol 5.connector.interconnect:CONN_01X04_MALE
- added J6: CONN_02X10, project_footprints:MOLEX_2035642017, symbol 5.connector.interconnect:CONN_02X10
- added Q5: Q_PMOS_GSD, 1_Semi_TO_SOT:TO-252-2, symbol 1.semi.discrete:Q_PMOS_GSD
- J2, J3, J8: footprint (none) -> project_footprints:JST_SM04B-GHS-TB(LF)(SN)-
- J4: footprint (none) -> project_footprints:JST_SM02B_GHS_TB
- R10, R8: PN 1,12 -> (none)
- U1: Link https://www.digikey.com/en/products/detail/samtec-inc/FTSH-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 -> (none); PN 5,5 -> (none)
- U10: PN 5,9 -> (none)
- U5: footprint (none) -> project_footprints:AMASS_XT30PW-M
Connections:
- net +3V3: now also J1.4, J5.4
- net +BATT: now also Q5.2 (S)
- net CAN_H: now also J5.3
- net CAN_L: now also J5.2
- net GND: now also U5.1 (-), J1.1, J5.1, Q5.1 (G)
- net RX: now also J1.2
- net SCL0: now also J8.2; no longer J2.2
- net SCL1: now also J2.2; no longer J8.2
- net SDA0: now also J8.3; no longer J2.3
- net SDA1: now also J2.3; no longer J8.3
- net TX: now also J1.3
- net USB_D+: now also U10.A6 (D+), U10.B6 (D+)
- net USB_D-: now also U10.A7 (D-), U10.B7 (D-)
- net at U5.2 (+): now also F1.1
- new net: F1.2, Q5.3 (D)
- new net CHAN_0A_OUT: J6.1 (P1)
- new net CHAN_0B_OUT: J6.2 (P2)
- new net CHAN_1A_OUT: J6.3 (P3)
- new net CHAN_1B_OUT: J6.4 (P4)
- new net CHAN_2A_OUT: J6.5 (P5)
- new net CHAN_2B_OUT: J6.6 (P6)
- new net CHAN_3A_OUT: J6.7 (P7)
- new net CHAN_3B_OUT: J6.8 (P8)
- new net CHAN_4A_OUT: J6.9 (P9)
- new net CHAN_4B_OUT: J6.10 (P10)
- new net CHAN_5A_OUT: J6.11 (P11)
- new net CHAN_5B_OUT: J6.12 (P12)
- new net CHAN_6A_OUT: J6.13 (P13)
- new net CHAN_6B_OUT: J6.14 (P14)
- new net CHAN_7A_OUT: J6.15 (P15)
- new net CHAN_7B_OUT: J6.16 (P16)
- no-connect marks 4 -> 8
Other:
- sheet peripherals ports: added ENC_BUTTON, ROT_ENC_A, ROT_ENC_B, SCL1, SDA1, TFT_DC; removed BUTTON_1, BUTTON_2, SCL0, SDA0, TFT_RESET
- sheet processor ports: added BUZZER, ENC_CTL_0, ENC_CTL_1, ENC_CTL_2, MISO0, MOSI0, ROT_ENC_A, ROT_ENC_B, SCK0, SD_CS, TFT_CS, TFT_DC; removed ECN_CTL_0, ECN_CTL_1, ECN_CTL_2, ECN_CTL_3, MISO, MOSI, SCK
- sheet switch_control ports: added none; removed ECN_CTL_3
- note added: "Battery Power (1-4S LIPO)"
- note added: "eOPRA Output"
- note removed: "Battery PoweR (1-4S LIPO)"
- moved on the sheet: J4, J8, R10, R8, TP3, U1, U10, U27, U28, U5, U7, U8

Commit message: Version updates
Other:
- company: (none) -> Massachusetts Institute of Technology / MIT Media Lab
- title: (none) -> eOPRA Switch / Stimulation Controller
- moved on the sheet: J1, J5, J8

Commit message: starting layout
Connections:
- net A_IN_0 is gone; now on net +3V3: J3.1
- net A_IN_1 is gone; now on net A_IN_2: J3.2
- net A_IN_2: no longer J3.3
- net A_IN_3: now also J3.3; no longer J3.4
- net GND: now also J3.4
Other:
- sheet peripherals ports: added ROT_ENC_0, ROT_ENC_1; removed ROT_ENC_A, ROT_ENC_B
- sheet processor ports: added ROT_ENC_0, ROT_ENC_1; removed A_IN_0, A_IN_1, ROT_ENC_A, ROT_ENC_B
- moved on the sheet: J1, J3, J4, J5, J6, J8

Commit message: before esp
Parts:
- added R13, R14: 27.4, 2_Passives_Resistors_SMD_IPC:R_1005_402_A, symbol 2.passive:R
Connections:
- net USB_D+: now also R14.2; no longer U10.A6 (D+), U10.B6 (D+)
- net USB_D-: now also R13.2; no longer U10.A7 (D-), U10.B7 (D-)
- new net: R14.1, U10.A6 (D+), U10.B6 (D+)
- new net: R13.1, U10.A7 (D-), U10.B7 (D-)
Other:
- note added: "Place termination resistors close to RP2040"
Changed lines of the file:
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@@
   (junction (at 28.575 61.595) (diameter 0) (color 0 0 0 0)
   )
+  (junction (at 46.99 40.64) (diameter 0) (color 0 0 0 0)
+  )
   (junction (at 46.99 27.94) (diameter 0) (color 0 0 0 0)
   )
@@
   (junction (at 36.195 61.595) (diameter 0) (color 0 0 0 0)
   )
+  (junction (at 64.135 189.865) (diameter 0) (color 0 0 0 0)
+  )
+  (junction (at 46.99 30.48) (diameter 0) (color 0 0 0 0)
+  )
+  (junction (at 26.67 83.185) (diameter 0) (color 0 0 0 0)
+  )
+  (junction (at 53.34 61.595) (diameter 0) (color 0 0 0 0)
+  )
+  (junction (at 31.115 61.595) (diameter 0) (color 0 0 0 0)
+  )
   (junction (at 46.99 35.56) (diameter 0) (color 0 0 0 0)
-  )
-  (junction (at 64.135 189.865) (diameter 0) (color 0 0 0 0)
-  )
-  (junction (at 46.99 30.48) (diameter 0) (color 0 0 0 0)
-  )
-  (junction (at 26.67 83.185) (diameter 0) (color 0 0 0 0)
-  )
-  (junction (at 53.34 61.595) (diameter 0) (color 0 0 0 0)
-  )
-  (junction (at 46.99 40.64) (diameter 0) (color 0 0 0 0)
-  )
-  (junction (at 31.115 61.595) (diameter 0) (color 0 0 0 0)
   )
   (no_connect (at 236.22 116.205))
@@
     (stroke (width 0) (type default))
   )
-  (wire (pts (xy 106.045 187.96) (xy 106.045 190.5))
-    (stroke (width 0) (type default))
-  )
   (wire (pts (xy 123.825 112.395) (xy 140.97 112.395))
     (stroke (width 0) (type default))
@@
     (stroke (width 0) (type default))
   )
+  (wire (pts (xy 46.99 40.64) (xy 47.625 40.64))
+    (stroke (width 0) (type default))
+  )
   (bus (pts (xy 143.51 121.92) (xy 143.51 123.825))
     (stroke (width 0) (type default))
@@
     (stroke (width 0) (type default))
   )
+  (wire (pts (xy 55.245 40.64) (xy 66.675 40.64))
+    (stroke (width 0) (type default))
+  )
+  (wire (pts (xy 55.245 35.56) (xy 66.675 35.56))
+    (stroke (width 0) (type default))
+  )
   (wire (pts (xy 250.825 100.965) (xy 248.92 100.965))
     (stroke (width 0) (type default))
@@
     (stroke (width 0) (type default))
   )
+  (wire (pts (xy 46.99 35.56) (xy 47.625 35.56))
+    (stroke (width 0) (type default))
+  )
   (wire (pts (xy 146.05 24.13) (xy 160.655 24.13))
     (stroke (width 0) (type default))
@@
     (stroke (width 0) (type default))
   )
-  (wire (pts (xy 46.99 40.64) (xy 66.675 40.64))
-    (stroke (width 0) (type default))
-  )
   (wire (pts (xy 154.305 58.42) (xy 154.94 58.42))
     (stroke (width 0) (type default))
@@
   )
   (wire (pts (xy 146.05 186.69) (xy 154.94 186.69))
-    (stroke (width 0) (type default))
-  )
-  (wire (pts (xy 46.99 35.56) (xy 66.675 35.56))
     (stroke (width 0) (type default))
   )
@@
     (fill (type none))
     (effects (font (size 1.27 1.27)) (justify left top))
+  )
+  (text "Place termination resistors \nclose to RP2040\n" (at 69.85 40.64 0)
+    (effects (font (size 1.27 1.27)) (justify left bottom))
   )
   (text "eOPRA Output\n" (at 230.505 87.63 0)
@@
         (path "/9f7a57db-2daa-452d-a1aa-74a4ad8115df"
           (reference "#PWR093") (unit 1)
+        )
+      )
+    )
+  )
+  (symbol (lib_id "2.passive:R") (at 51.435 40.64 90) (unit 1)
+    (in_bom yes) (on_board yes) (dnp no)
+    (property "Reference" "R14" (at 49.53 43.18 90)
+      (effects (font (size 1.27 1.27)))
+    )
+    (property "Value" "27.4" (at 54.61 43.18 90)
+      (effects (font (size 1.27 1.27)))
+    )
+    (property "Footprint" "2_Passives_Resistors_SMD_IPC:R_1005_402_A" (at 51.435 42.418 90)
+      (effects (font (size 1.27 1.27)) hide)
+    )
+    (property "Datasheet" "~" (at 51.435 40.64 0)
+      (effects (font (size 1.27 1.27)) hide)
+    )
+    (pin "1")
+    (pin "2")
+    (instances
+      (project "eOPRA_interface"
+        (path "/9f7a57db-2daa-452d-a1aa-74a4ad8115df"
+          (reference "R14") (unit 1)
+        )
+        (path "/9f7a57db-2daa-452d-a1aa-74a4ad8115df/d165d604-1acf-4179-9574-6e327e7130e7"
+          (reference "R14") (unit 1)
         )
       )
@@
     )
   )
+  (symbol (lib_id "2.passive:R") (at 51.435 35.56 90) (unit 1)
+    (in_bom yes) (on_board yes) (dnp no)
+    (property "Reference" "R13" (at 49.53 38.1 90)
+      (effects (font (size 1.27 1.27)))
+    )
+    (property "Value" "27.4" (at 54.61 38.1 90)
+      (effects (font (size 1.27 1.27)))
+    )
+    (property "Footprint" "2_Passives_Resistors_SMD_IPC:R_1005_402_A" (at 51.435 37.338 90)
+      (effects (font (size 1.27 1.27)) hide)
+    )
+    (property "Datasheet" "~" (at 51.435 35.56 0)
+      (effects (font (size 1.27 1.27)) hide)
+    )
+    (pin "1")
+    (pin "2")
+    (instances
+      (project "eOPRA_interface"
+        (path "/9f7a57db-2daa-452d-a1aa-74a4ad8115df"
+          (reference "R13") (unit 1)
+        )
+        (path "/9f7a57db-2daa-452d-a1aa-74a4ad8115df/d165d604-1acf-4179-9574-6e327e7130e7"
+          (reference "R13") (unit 1)
+        )
+      )
+    )
+  )
   (symbol (lib_id "5.connector.interconnect:CONN_01X04_MALE") (at 162.56 184.15 180) (unit 1)
     (in_bom yes) (on_board yes) (dnp no)
@@
     )
   )
-  (symbol (lib_id "0.power-symbols:+3.3V") (at 106.045 187.96 0) (unit 1)
-    (in_bom yes) (on_board yes) (dnp no) (fields_autoplaced)
-    (property "Reference" "#PWR06" (at 106.045 191.77 0)
-      (effects (font (size 1.27 1.27)) hide)
-    )
-    (property "Value" "+3.3V" (at 106.045 184.4581 0)
-      (effects (font (size 1.27 1.27)))
-    )
-    (property "Footprint" "" (at 106.045 187.96 0)
-      (effects (font (size 1.27 1.27)) hide)
-    )
-    (property "Datasheet" "" (at 106.045 187.96 0)
-      (effects (font (size 1.27 1.27)) hide)
-    )
-    (pin "1")
-    (instances
-      (project "eOPRA_interface"
-        (path "/9f7a57db-2daa-452d-a1aa-74a4ad8115df"
-          (reference "#PWR06") (unit 1)
-        )
-      )
-    )
-  )
   (symbol (lib_id "5.connector.interconnect:CONN_01X04_MALE") (at 162.56 130.81 180) (unit 1)
     (in_bom yes) (on_board yes) (dnp no)
@@
         )
       )
-    )
-  )
-  (symbol (lib_id "0.power-symbols:PWR_FLAG") (at 106.045 190.5 180) (unit 1)
-    (in_bom yes) (on_board yes) (dnp no) (fields_autoplaced)
-    (property "Reference" "#FLG04" (at 106.045 192.405 0)
-      (effects (font (size 1.27 1.27)) hide)
-    )
-    (property "Value" "PWR_FLAG" (at 106.045 194.6355 0)
-      (effects (font (size 1.27 1.27)))
-    )
-    (property "Footprint" "" (at 106.045 190.5 0)
-      (effects (font (size 1.27 1.27)) hide)
-    )
-    (property "Datasheet" "" (at 106.045 190.5 0)
-      (effects (font (size 1.27 1.27)) hide)
-    )
-    (pin "1")
-    (instances
-      (project "eOPRA_interface"
-        (path "/9f7a57db-2daa-452d-a1aa-74a4ad8115df"
-          (reference "#FLG04") (unit 1)
-        )
-      )

Commit message: before 4 layer
Parts:
- removed TP3: TEST, 0_misc:test_point_2mm_square, symbol 5.connector.interconnect:TEST
Connections:
- net GNDD is gone; now on net GND: R10.2, R8.1, U1.3 (GND), U1.5 (GND), U10.A1 (GND), U10.A12 (GND), U10.B1 (GND), U10.B12 (GND), U10.S1 (SHIELD)
- no-connect marks 8 -> 9
Changed lines of the file:
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@@
   (no_connect (at 248.92 116.205))
   (no_connect (at 56.515 85.725))
+  (no_connect (at 28.575 88.265))
   (no_connect (at 46.355 53.34))
   (no_connect (at 56.515 83.185))
@@
     (stroke (width 0) (type default))
   )
-  (wire (pts (xy 24.765 88.265) (xy 28.575 88.265))
-    (stroke (width 0) (type default))
-  )
   (bus (pts (xy 143.51 41.91) (xy 143.51 43.815))
     (stroke (width 0) (type default))
@@
     )
   )
-  (symbol (lib_id "0.power-symbols:GNDD") (at 53.34 64.135 0) (mirror y) (unit 1)
-    (in_bom yes) (on_board yes) (dnp no) (fields_autoplaced)
-    (property "Reference" "#PWR03" (at 53.34 70.485 0)
-      (effects (font (size 1.27 1.27)) hide)
-    )
-    (property "Value" "GNDD" (at 53.34 68.5784 0)
-      (effects (font (size 1.27 1.27)))
-    )
-    (property "Footprint" "" (at 53.34 64.135 0)
-      (effects (font (size 1.27 1.27)) hide)
-    )
-    (property "Datasheet" "" (at 53.34 64.135 0)
-      (effects (font (size 1.27 1.27)) hide)
-    )
-    (pin "1")
-    (instances
-      (project "1.0"
-        (path "/628082f8-0394-4f00-be88-5631e8394d3a"
-          (reference "#PWR03") (unit 1)
-        )
-      )
-      (project "eOPRA_interface"
-        (path "/9f7a57db-2daa-452d-a1aa-74a4ad8115df"
-          (reference "#PWR03") (unit 1)
-        )
-      )
-    )
-  )
   (symbol (lib_id "2.passive:R") (at 50.165 56.515 180) (unit 1)
     (in_bom yes) (on_board yes) (dnp no)
@@
         (path "/9f7a57db-2daa-452d-a1aa-74a4ad8115df"
           (reference "Q5") (unit 1)
-        )
-      )
-    )
-  )
-  (symbol (lib_id "0.power-symbols:GNDD") (at 26.67 90.17 0) (mirror y) (unit 1)
-    (in_bom yes) (on_board yes) (dnp no) (fields_autoplaced)
-    (property "Reference" "#PWR02" (at 26.67 96.52 0)
-      (effects (font (size 1.27 1.27)) hide)
-    )
-    (property "Value" "GNDD" (at 26.67 94.6134 0)
-      (effects (font (size 1.27 1.27)))
-    )
-    (property "Footprint" "" (at 26.67 90.17 0)
-      (effects (font (size 1.27 1.27)) hide)
-    )
-    (property "Datasheet" "" (at 26.67 90.17 0)
-      (effects (font (size 1.27 1.27)) hide)
-    )
-    (pin "1")
-    (instances
-      (project "1.0"
-        (path "/628082f8-0394-4f00-be88-5631e8394d3a"
-          (reference "#PWR02") (unit 1)
-        )
-      )
-      (project "eOPRA_interface"
-        (path "/9f7a57db-2daa-452d-a1aa-74a4ad8115df"
-          (reference "#PWR02") (unit 1)
         )
       )
@@
     )
   )
+  (symbol (lib_id "0.power-symbols:GND") (at 26.67 90.17 0) (unit 1)
+    (in_bom yes) (on_board yes) (dnp no) (fields_autoplaced)
+    (property "Reference" "#PWR02" (at 26.67 96.52 0)
+      (effects (font (size 1.27 1.27)) hide)
+    )
+    (property "Value" "GND" (at 26.67 94.3055 0)
+      (effects (font (size 1.27 1.27)))
+    )
+    (property "Footprint" "" (at 26.67 90.17 0)
+      (effects (font (size 1.27 1.27)) hide)
+    )
+    (property "Datasheet" "" (at 26.67 90.17 0)
+      (effects (font (size 1.27 1.27)) hide)
+    )
+    (pin "1")
+    (instances
+      (project "eOPRA_interface"
+        (path "/9f7a57db-2daa-452d-a1aa-74a4ad8115df"
+          (reference "#PWR02") (unit 1)
+        )
+      )
+    )
+  )
   (symbol (lib_id "0.power-symbols:GND") (at 85.09 190.5 0) (unit 1)
     (in_bom yes) (on_board yes) (dnp no) (fields_autoplaced)
@@
     )
   )
+  (symbol (lib_id "0.power-symbols:GND") (at 53.34 64.135 0) (unit 1)
+    (in_bom yes) (on_board yes) (dnp no) (fields_autoplaced)
+    (property "Reference" "#PWR06" (at 53.34 70.485 0)
+      (effects (font (size 1.27 1.27)) hide)
+    )
+    (property "Value" "GND" (at 53.34 68.2705 0)
+      (effects (font (size 1.27 1.27)))
+    )
+    (property "Footprint" "" (at 53.34 64.135 0)
+      (effects (font (size 1.27 1.27)) hide)
+    )
+    (property "Datasheet" "" (at 53.34 64.135 0)
+      (effects (font (size 1.27 1.27)) hide)
+    )
+    (pin "1")
+    (instances
+      (project "eOPRA_interface"
+        (path "/9f7a57db-2daa-452d-a1aa-74a4ad8115df"
+          (reference "#PWR06") (unit 1)
+        )
+      )
+    )
+  )
   (symbol (lib_id "5.connector.interconnect:CONN_01X04_MALE") (at 162.56 66.04 180) (unit 1)
     (in_bom yes) (on_board yes) (dnp no)
@@
         )
       )
-    )
-  )
-  (symbol (lib_id "5.connector.interconnect:TEST") (at 24.765 88.265 90) (unit 1)
-    (in_bom yes) (on_board yes) (dnp no)
-    (property "Reference" "TP3" (at 15.875 90.17 0)
-      (effects (font (size 1.27 1.27)) (justify left))
-    )
-    (property "Value" "TEST" (at 18.4119 90.17 0)
-      (effects (font (size 1.27 1.27)) (justify left))
-    )
-    (property "Footprint" "0_misc:test_point_2mm_square" (at 24.765 88.265 0)
-      (effects (font (size 1.27 1.27)) hide)
-    )
-    (property "Datasheet" "" (at 24.765 88.265 0)
-      (effects (font (size 1.27 1.27)) hide)
-    )
-    (pin "1")
-    (instances
-      (project "1.0"
-        (path "/628082f8-0394-4f00-be88-5631e8394d3a/94532174-4d89-478b-a3e8-1052be6253fa"
-          (reference "TP3") (unit 1)
-        )
-        (path "/628082f8-0394-4f00-be88-5631e8394d3a"
-          (reference "TP2") (unit 1)
-        )
-      )
-      (project "eOPRA_interface"
-        (path "/9f7a57db-2daa-452d-a1aa-74a4ad8115df"
-          (reference "TP1") (unit 1)
-        )
-      )

Commit message: preliminary finish
Changed lines of the file:
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@@
-    (stroke (width 0) (type default))
-  )
-  (wire (pts (xy 85.09 187.96) (xy 85.09 190.5))
     (stroke (width 0) (type default))
   )
@@
     )
   )
-  (symbol (lib_id "0.power-symbols:GND") (at 85.09 190.5 0) (unit 1)
-    (in_bom yes) (on_board yes) (dnp no) (fields_autoplaced)
-    (property "Reference" "#PWR0108" (at 85.09 196.85 0)
-      (effects (font (size 1.27 1.27)) hide)
-    )
-    (property "Value" "GND" (at 85.09 194.6355 0)
-      (effects (font (size 1.27 1.27)))
-    )
-    (property "Footprint" "" (at 85.09 190.5 0)
-      (effects (font (size 1.27 1.27)) hide)
-    )
-    (property "Datasheet" "" (at 85.09 190.5 0)
-      (effects (font (size 1.27 1.27)) hide)
-    )
-    (pin "1")
-    (instances
-      (project "eOPRA_interface"
-        (path "/9f7a57db-2daa-452d-a1aa-74a4ad8115df"
-          (reference "#PWR0108") (unit 1)
-        )
-      )
-    )
-  )
   (symbol (lib_id "0.power-symbols:PWR_FLAG") (at 94.615 190.5 180) (unit 1)
     (in_bom yes) (on_board yes) (dnp no) (fields_autoplaced)
@@
         )
       )
-    )
-  )
-  (symbol (lib_id "0.power-symbols:PWR_FLAG") (at 85.09 187.96 0) (unit 1)
-    (in_bom yes) (on_board yes) (dnp no) (fields_autoplaced)
-    (property "Reference" "#FLG03" (at 85.09 186.055 0)
-      (effects (font (size 1.27 1.27)) hide)
-    )
-    (property "Value" "PWR_FLAG" (at 85.09 184.4581 0)
-      (effects (font (size 1.27 1.27)))
-    )
-    (property "Footprint" "" (at 85.09 187.96 0)
-      (effects (font (size 1.27 1.27)) hide)
-    )
-    (property "Datasheet" "" (at 85.09 187.96 0)
-      (effects (font (size 1.27 1.27)) hide)
-    )
-    (pin "1")
-    (instances
-      (project "eOPRA_interface"
-        (path "/9f7a57db-2daa-452d-a1aa-74a4ad8115df"
-          (reference "#FLG03") (unit 1)
-        )
-      )

Commit message: draft 2 wifi finish
Parts:
- added J7: CONN_01X04_MALE, project_footprints:JST_SM04B-GHS-TB(LF)(SN)-, symbol 5.connector.interconnect:CONN_01X04_MALE
- added TP9: TEST, 0_misc:test_point_1.0mm_square, symbol 5.connector.interconnect:TEST
Connections:
- net GND: now also J7.4
- new net: J7.1, TP9.1
- new net RXD: J7.2
- new net TXD: J7.3
Other:
- added sheet ESP-Wifi (ESP-Wifi.kicad_sch)
- sheet processor ports: added ESP_INT; removed none
- moved on the sheet: F1, J1, J2, J3, J4, J5, J6, J8, Q5, R10, R13, R14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

Commit message: stuff
Parts:
- removed R13, R14: 27.4, 2_Passives_Resistors_SMD_IPC:R_1005_402_A, symbol 2.passive:R
- removed TP9: TEST, 0_misc:test_point_1.0mm_square, symbol 5.connector.interconnect:TEST
- added D2: D_Schottky, 1_Semi_Discrete_Diodes_SMD:D_SOD-123F, symbol 1.semi.discrete:D_Schottky
- added TP5 (x2): TEST, 0_misc:test_point_0.8mm_square, symbol 5.connector.interconnect:TEST
- F1: PN (none) -> 5,1
- J1, J2, J3, J5, J7, J8: PN (none) -> 8,1
- J4: PN (none) -> 8,2
- J6: PN (none) -> 8,3
- Q5: footprint 1_Semi_TO_SOT:TO-252-2 -> project_footprints:SON_8DU-T1-GE3_VIS; PN (none) -> 10,3
- R10, R8: PN (none) -> 1,1
- U1: PN (none) -> 8,5
- U10: PN (none) -> 8,6
- U5: PN (none) -> 8,4
Connections:
- net +3V3: now also D2.1 (K)
- net EMG_HIGH: now also TP5.1
- net EMG_LOW: now also TP5.1
- net USB_D+: now also U10.A6 (D+), U10.B6 (D+)
- net USB_D-: now also U10.A7 (D-), U10.B7 (D-)
- net at J7.1: now also D2.2 (A)
Other:
- note added: "CHECK FET"
- note removed: "Place termination resistors close to RP2040"
- moved on the sheet: J6, U27, U28, U7, U8
