File: eOPRA_interface/processor.kicad_sch (KiCad schematic)
At the start: 38 parts, among them SW2 SW_Push, SW6 SW_Push, U10 RP2040, U11 W25Q128JVS, U13 MCP25625, Y1 12Mhz 12pF, Y2 16Mhz 12pF

Commit message: schematic v1.0 finished
Parts:
- removed R97, R98 (x2): 4k7, 2_Passives_Resistors_SMD_IPC:R_1608_603_B, symbol 2.passive:R
- removed SW2, SW6: SW_Push, symbol 3.electromechanical.switch:SW_Push
- removed Y1: 12Mhz 12pF, symbol 2.passive:Crystal
- removed Y2: 16Mhz 12pF, symbol 2.passive:Crystal
- added C25: 100nF, 2_Passives_Capacitors_SMD_IPC:C_1005_402_A, symbol 2.passive:C
- added D2, D7, D8, D9: D_Zener, project_footprints:SOD-323, symbol 1.semi.discrete:D_Zener
- added D6: WS2812B, 1_Semi_LED-Opto:WS2812B, symbol 1.semi.opto:WS2812B
- added R11, R22, R24, R27, R28: 10k, 2_Passives_Resistors_SMD_IPC:R_1608_603_B, symbol 2.passive:R
- added R81: 500, 2_Passives_Resistors_SMD_IPC:R_1005_402_A, symbol 2.passive:R
- added R97 (x3): 4k7, 2_Passives_Resistors_SMD_IPC:R_1608_603_B, symbol 2.passive:R
- added SW1 (x2): SW_Push, project_footprints:TL3365AF180QG, symbol 3.electromechanical.switch:SW_Push
- added TP3: TEST, 0_misc:test_point_2mm_square, symbol 5.connector.interconnect:TEST
- added Y1: 16Mhz 12pF, project_footprints:4-smd, symbol 2.passive:Crystal_GND24
- added Y3: 12Mhz 12pF, project_footprints:4-smd, symbol 2.passive:Crystal_GND24
- C10, C11, C12, C13, C14, C15, C7, C8, C9: footprint (none) -> 2_Passives_Capacitors_SMD_IPC:C_1005_402_A
- C16, C17, C21, C22, C23, C24, R4: footprint (none) -> 2_Passives_Resistors_SMD_IPC:R_1005_402_A
- C4, C5: value C -> 22pF; footprint (none) -> 2_Passives_Resistors_SMD_IPC:R_1005_402_A
- D1: footprint 1_Semi_TO_SOT:TSOT-23 -> 1_Semi_TO_SOT:SOT-23
- D3: footprint (none) -> 1_Semi_Discrete_Diodes_SMD:D_0603
- R11, R12: value R -> 27.4; footprint (none) -> 2_Passives_Resistors_SMD_IPC:R_1005_402_A
- R15: footprint (none) -> 2_Passives_Resistors_SMD_IPC:R_1608_603_B
- R16, R17: value R -> 500; footprint (none) -> 2_Passives_Resistors_SMD_IPC:R_1608_603_B
- R25: value R -> 10k; footprint (none) -> 2_Passives_Resistors_SMD_IPC:R_1608_603_B
- R97: PN 1,6 -> (none)
- U10: footprint (none) -> project_footprints:QFN40P700X700X90-57N
- U11: footprint (none) -> 1_Semi_Misc:GD25Q16CWIGR
Connections:
- net USB_BOOT is gone; now on net QSPI_CS: R17.2
- net +1V1: no longer U10.44 (VREG_IN)
- net +3V3: now also U10.44 (VREG_VIN), C25.1, D6.1 (VDD), R11.2, R97.2, R97.2, R97.2
- net A_IN_0: now also D2.1 (K), R22.1, R22.2; no longer U10.38 (GPIO26_ADC0)
- net A_IN_1: now also D7.1 (K), R24.1, R24.2; no longer U10.39 (GPIO27_ADC1)
- net A_IN_2: now also D8.1 (K), R27.1, R27.2
- net A_IN_3: now also D9.1 (K), R28.1, R28.2
- net CAN_CS: now also R11.1
- net CAN_RESET: now also R25.2, U13.2 (~{RESET})
- net CAN_STBY: now also R15.1, U13.15 (STBY)
- net GND: now also C21.2, C5.2, U13.29 (EP), C25.2, D2.2 (A), D6.3 (GND), D7.2 (A), D8.2 (A), D9.2 (A), SW1.2, SW1.2, SW1.4, SW1.4, Y1.2, Y1.4, Y3.2, Y3.4; no longer C21.1, C5.1
- net SCL0: now also U10.32 (GPIO21), R97.1; no longer U10.7 (GPIO5)
- net SCL1: now also U10.39 (GPIO27_ADC1), R97.1; no longer U10.5 (GPIO3)
- net SDA0: now also U10.31 (GPIO20); no longer U10.6 (GPIO4)
- net SDA1: now also U10.38 (GPIO26_ADC0), R97.1; no longer U10.4 (GPIO2)
- net ~{RESET}: now also SW1.1, SW1.3
- net at R4.1: now also C5.1, Y3.1; no longer C5.2
- net at C4.2, U10.20 (XIN): now also Y3.3
- net at U13.20 (OSC2): now also R81.2; no longer C21.2
- net at C22.2, U13.21 (OSC1): now also Y1.3
- net at D3.1 (K): now also SW1.1, SW1.3
- net MISO renamed MISO1
- net MISO1: now also U10.15 (GPIO12); no longer U10.11 (GPIO8)
- net MOSI renamed ENC_CTL_2
- net ENC_CTL_2: no longer U13.27 (MOSI)
- removed net OPEN: U10.12 (GPIO9), U10.13 (GPIO10), U10.14 (GPIO11), U10.15 (GPIO12), U10.16 (GPIO13), U10.31 (GPIO20), U10.32 (GPIO21), U10.36 (GPIO24), U10.37 (GPIO25), U10.8 (GPIO6)
- net PIN_BUTTON - UNSP renamed SD_CS
- net SCK renamed ENC_CTL_1
- net ENC_CTL_1: no longer U13.26 (SCK)
- new net: C21.1, R81.1, Y1.1
- new net BUZZER: U10.8 (GPIO6)
- new net ENC_CTL_0: U10.16 (GPIO13)
- new net LED_CTL: D6.4 (DIN), U10.7 (GPIO5)
- new net MISO0: U10.6 (GPIO4)
- new net MOSI0: U10.5 (GPIO3)
- new net MOSI1: U10.14 (GPIO11), U13.27 (MOSI)
- new net ROT_ENC_A: U10.36 (GPIO24)
- new net ROT_ENC_B: U10.37 (GPIO25)
- new net SCK0: U10.4 (GPIO2)
- new net SCK1: U10.13 (GPIO10), U13.26 (SCK)
- new net TFT_CS: TP3.1, U10.12 (GPIO9)
- new net TFT_DC: U10.11 (GPIO8)
- no-connect marks 3 -> 5
Other:
- note added: "(RP2040 ~{CS})"
- note added: "(System) Flash"
- note added: "Analog In protection"
- note added: "Place close to DVDDs"
- note added: "Place close to VREG_VOUT and VREG_VIN"
- moved on the sheet: C22, C23, C24, D1, D3, R15, R17, R25, R4, R97

Commit message: Version updates
Other:
- company: (none) -> Massachusetts Institute of Technology / MIT Media Lab
- title: (none) -> eOPRA Switch / Stimulation Controller
Changed lines of the file:
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@@
 (kicad_sch (version 20230121) (generator eeschema)
   (paper "A3")
+  (title_block
+    (title "eOPRA Switch / Stimulation Controller")
+    (date "2023-08-01")
+    (rev "1.0")
+    (company "Massachusetts Institute of Technology / MIT Media Lab")
+  )
   (junction (at 223.52 55.245) (diameter 0) (color 0 0 0 0)
   )

Commit message: starting layout
Parts:
- removed D2, D7: D_Zener, project_footprints:SOD-323, symbol 1.semi.discrete:D_Zener
- removed R22, R24: 10k, 2_Passives_Resistors_SMD_IPC:R_1608_603_B, symbol 2.passive:R
Connections:
- net BUZZER: now also U10.11 (GPIO8); no longer U10.8 (GPIO6)
- net LED_CTL: now also U10.9 (GPIO7); no longer U10.7 (GPIO5)
- net SD_CS: now also U10.8 (GPIO6); no longer U10.9 (GPIO7)
- net TFT_DC: now also U10.7 (GPIO5); no longer U10.11 (GPIO8)
- net ROT_ENC_A renamed ROT_ENC_0
- net ROT_ENC_B renamed ROT_ENC_1
Other:
- moved on the sheet: D8, D9, R27, R28, TP3

Commit message: before esp
Parts:
- removed R11, R12: 27.4, 2_Passives_Resistors_SMD_IPC:R_1005_402_A, symbol 2.passive:R
- R16: now not fitted
- R17: value 500 -> 1k; footprint 2_Passives_Resistors_SMD_IPC:R_1608_603_B -> 2_Passives_Resistors_SMD_IPC:R_1005_402_A
Connections:
- net QSPI_CS: now also R17.1; no longer R17.2
- net USB_D+: now also U10.47 (USB_D+)
- net USB_D-: now also U10.46 (USB_D-)
- net at D3.2 (A): now also R17.2; no longer R17.1
Other:
- note removed: "Place termination resistors close to RP2040"
Changed lines of the file:
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@@
+    (stroke (width 0) (type default))
+  )
+  (wire (pts (xy 158.115 114.3) (xy 160.02 114.3))
     (stroke (width 0) (type default))
   )
@@
     (stroke (width 0) (type default))
   )
-  (wire (pts (xy 158.75 114.3) (xy 160.02 114.3))
-    (stroke (width 0) (type default))
-  )
   (wire (pts (xy 139.7 152.4) (xy 140.335 152.4))
     (stroke (width 0) (type default))
@@
     (stroke (width 0) (type default))
   )
+  (wire (pts (xy 158.115 108.585) (xy 160.02 108.585))
+    (stroke (width 0) (type default))
+  )
   (wire (pts (xy 52.07 264.16) (xy 52.07 261.62))
     (stroke (width 0) (type default))
@@
     (stroke (width 0) (type default))
   )
-  (wire (pts (xy 140.97 108.585) (xy 142.24 108.585))
-    (stroke (width 0) (type default))
-  )
   (wire (pts (xy 36.83 264.16) (xy 36.83 261.62))
     (stroke (width 0) (type default))
@@
     (stroke (width 0) (type default))
   )
-  (wire (pts (xy 149.86 108.585) (xy 160.02 108.585))
-    (stroke (width 0) (type default))
-  )
   (wire (pts (xy 306.07 107.315) (xy 306.07 108.585))
     (stroke (width 0) (type default))
@@
   )
   (wire (pts (xy 165.1 241.935) (xy 163.83 241.935))
-    (stroke (width 0) (type default))
-  )
-  (wire (pts (xy 140.97 114.3) (xy 151.13 114.3))
     (stroke (width 0) (type default))
   )
@@
     (effects (font (size 3 3)) (justify left bottom))
   )
-  (text "Place termination resistors \nclose to RP2040\n" (at 105.41 112.395 0)
-    (effects (font (size 1.27 1.27)) (justify left bottom))
-  )
   (text "Boot / Reset Buttons\n" (at 31.115 231.775 0)
     (effects (font (size 3 3)) (justify left bottom))
@@
     (effects (font (size 1.27 1.27)) (justify left bottom))
   )
-  (hierarchical_label "USB_D+" (shape bidirectional) (at 140.97 108.585 180) (fields_autoplaced)
+  (hierarchical_label "USB_D+" (shape bidirectional) (at 158.115 108.585 180) (fields_autoplaced)
     (effects (font (size 1.27 1.27)) (justify right))
   )
@@
     (effects (font (size 1.27 1.27)) (justify left))
   )
-  (hierarchical_label "USB_D-" (shape bidirectional) (at 140.97 114.3 180) (fields_autoplaced)
+  (hierarchical_label "USB_D-" (shape bidirectional) (at 158.115 114.3 180) (fields_autoplaced)
     (effects (font (size 1.27 1.27)) (justify right))
   )
@@
     )
   )
-  (symbol (lib_id "2.passive:R") (at 146.05 108.585 90) (unit 1)
-    (in_bom yes) (on_board yes) (dnp no)
-    (property "Reference" "R11" (at 145.415 106.045 90)
-      (effects (font (size 1.27 1.27)))
-    )
-    (property "Value" "27.4" (at 145.415 111.125 90)
-      (effects (font (size 1.27 1.27)))
-    )
-    (property "Footprint" "2_Passives_Resistors_SMD_IPC:R_1005_402_A" (at 146.05 110.363 90)
-      (effects (font (size 1.27 1.27)) hide)
-    )
-    (property "Datasheet" "~" (at 146.05 108.585 0)
-      (effects (font (size 1.27 1.27)) hide)
-    )
-    (pin "1")
-    (pin "2")
-    (instances
-      (project "eOPRA_interface"
-        (path "/9f7a57db-2daa-452d-a1aa-74a4ad8115df"
-          (reference "R11") (unit 1)
-        )
-        (path "/9f7a57db-2daa-452d-a1aa-74a4ad8115df/d165d604-1acf-4179-9574-6e327e7130e7"
-          (reference "R13") (unit 1)
-        )
-      )
-    )
-  )
   (symbol (lib_id "2.passive:R") (at 294.005 112.395 180) (unit 1)
     (in_bom yes) (on_board yes) (dnp no)
@@
     )
   )
+  (symbol (lib_id "2.passive:R") (at 36.83 244.475 0) (unit 1)
+    (in_bom yes) (on_board yes) (dnp no)
+    (property "Reference" "R17" (at 33.02 245.11 0)
+      (effects (font (size 1.27 1.27)))
+    )
+    (property "Value" "1k" (at 31.115 243.205 0)
+      (effects (font (size 1.27 1.27)) (justify left))
+    )
+    (property "Footprint" "2_Passives_Resistors_SMD_IPC:R_1005_402_A" (at 35.052 244.475 90)
+      (effects (font (size 1.27 1.27)) hide)
+    )
+    (property "Datasheet" "~" (at 36.83 244.475 0)
+      (effects (font (size 1.27 1.27)) hide)
+    )
+    (pin "1")
+    (pin "2")
+    (instances
+      (project "eOPRA_interface"
+        (path "/9f7a57db-2daa-452d-a1aa-74a4ad8115df/d165d604-1acf-4179-9574-6e327e7130e7"
+          (reference "R17") (unit 1)
+        )
+      )
+    )
+  )
   (symbol (lib_id "2.passive:R") (at 363.22 207.645 180) (unit 1)
     (in_bom yes) (on_board yes) (dnp no)
@@
     )
   )
-  (symbol (lib_id "2.passive:R") (at 154.94 114.3 90) (unit 1)
-    (in_bom yes) (on_board yes) (dnp no)
-    (property "Reference" "R12" (at 153.67 111.76 90)
-      (effects (font (size 1.27 1.27)))
-    )
-    (property "Value" "27.4" (at 154.305 116.84 90)
-      (effects (font (size 1.27 1.27)))
-    )
-    (property "Footprint" "2_Passives_Resistors_SMD_IPC:R_1005_402_A" (at 154.94 116.078 90)
-      (effects (font (size 1.27 1.27)) hide)
-    )
-    (property "Datasheet" "~" (at 154.94 114.3 0)
-      (effects (font (size 1.27 1.27)) hide)
-    )
-    (pin "1")
-    (pin "2")
-    (instances
-      (project "eOPRA_interface"
-        (path "/9f7a57db-2daa-452d-a1aa-74a4ad8115df"
-          (reference "R12") (unit 1)
-        )
-        (path "/9f7a57db-2daa-452d-a1aa-74a4ad8115df/d165d604-1acf-4179-9574-6e327e7130e7"
-          (reference "R14") (unit 1)
-        )
-      )
-    )
-  )
   (symbol (lib_id "0.power-symbols:+1V1") (at 129.54 41.275 0) (unit 1)
     (in_bom yes) (on_board yes) (dnp no) (fields_autoplaced)
@@
   )
   (symbol (lib_id "2.passive:R") (at 41.91 142.24 180) (unit 1)
-    (in_bom yes) (on_board yes) (dnp no)
+    (in_bom yes) (on_board yes) (dnp yes)
     (property "Reference" "R16" (at 36.195 141.589 0)
       (effects (font (size 1.27 1.27)) (justify right))
@@
         )
       )
-    )
-  )
-  (symbol (lib_id "2.passive:R") (at 36.83 244.475 180) (unit 1)
-    (in_bom yes) (on_board yes) (dnp no)
-    (property "Reference" "R17" (at 31.115 243.84 0)
-      (effects (font (size 1.27 1.27)) (justify right))
-    )
-    (property "Value" "500" (at 31.115 245.761 0)
-      (effects (font (size 1.27 1.27)) (justify right))
-    )
-    (property "Footprint" "2_Passives_Resistors_SMD_IPC:R_1608_603_B" (at 38.608 244.475 90)
-      (effects (font (size 1.27 1.27)) hide)
-    )
-    (property "Datasheet" "~" (at 36.83 244.475 0)
-      (effects (font (size 1.27 1.27)) hide)
-    )
-    (pin "1")
-    (pin "2")
-    (instances
-      (project "eOPRA_interface"
-        (path "/9f7a57db-2daa-452d-a1aa-74a4ad8115df/d165d604-1acf-4179-9574-6e327e7130e7"
-          (reference "R17") (unit 1)
-        )
-      )

Commit message: before 4 layer
Connections:
- net A_IN_2: no longer D8.1 (K), R27.2, U10.40 (GPIO28_ADC2)
- net A_IN_3: no longer D9.1 (K), R28.2, U10.41 (GPIO29_ADC3)
- new net A_IN_2_PIN: D8.1 (K), R27.2, U10.40 (GPIO28_ADC2)
- new net A_IN_3_PIN: D9.1 (K), R28.2, U10.41 (GPIO29_ADC3)
Other:
- moved on the sheet: D9, R28
Changed lines of the file:
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@@
   (junction (at 277.495 43.18) (diameter 0) (color 0 0 0 0)
   )
-  (junction (at 165.1 241.935) (diameter 0) (color 0 0 0 0)
+  (junction (at 167.64 241.935) (diameter 0) (color 0 0 0 0)
   )
   (junction (at 280.035 148.59) (diameter 0) (color 0 0 0 0)
@@
     (stroke (width 0) (type default))
   )
-  (wire (pts (xy 165.1 241.935) (xy 166.37 241.935))
+  (wire (pts (xy 167.64 241.935) (xy 168.91 241.935))
     (stroke (width 0) (type default))
   )
@@
     (stroke (width 0) (type default))
   )
-  (wire (pts (xy 165.1 243.205) (xy 165.1 241.935))
+  (wire (pts (xy 167.64 243.205) (xy 167.64 241.935))
     (stroke (width 0) (type default))
   )
@@
     (stroke (width 0) (type default))
   )
-  (wire (pts (xy 165.1 241.935) (xy 163.83 241.935))
+  (wire (pts (xy 167.64 241.935) (xy 166.37 241.935))
     (stroke (width 0) (type default))
   )
@@
     (stroke (width 0) (type default))
   )
-  (wire (pts (xy 154.94 241.935) (xy 156.21 241.935))
+  (wire (pts (xy 157.48 241.935) (xy 158.75 241.935))
     (stroke (width 0) (type default))
   )
@@
     (stroke (width 0) (type default))
   )
-  (wire (pts (xy 165.1 250.825) (xy 165.1 251.46))
+  (wire (pts (xy 167.64 250.825) (xy 167.64 251.46))
     (stroke (width 0) (type default))
   )
@@
     (effects (font (size 1.27 1.27)) (justify right bottom))
   )
+  (label "A_IN_2_PIN" (at 226.06 175.895 0) (fields_autoplaced)
+    (effects (font (size 1.27 1.27)) (justify left bottom))
+  )
   (label "QSPI_SD3" (at 80.01 154.305 0) (fields_autoplaced)
     (effects (font (size 1.27 1.27)) (justify left bottom))
@@
     (effects (font (size 1.27 1.27)) (justify right bottom))
   )
+  (label "A_IN_3_PIN" (at 168.91 241.935 0) (fields_autoplaced)
+    (effects (font (size 1.27 1.27)) (justify left bottom))
+  )
   (label "CAN_CS" (at 289.56 122.555 180) (fields_autoplaced)
     (effects (font (size 1.27 1.27)) (justify right bottom))
@@
     (effects (font (size 1.27 1.27)) (justify right bottom))
   )
-  (label "A_IN_2" (at 125.73 241.935 180) (fields_autoplaced)
-    (effects (font (size 1.27 1.27)) (justify right bottom))
+  (label "A_IN_2_PIN" (at 137.16 241.935 0) (fields_autoplaced)
+    (effects (font (size 1.27 1.27)) (justify left bottom))
   )
   (label "MISO1" (at 226.06 132.715 0) (fields_autoplaced)
@@
     (effects (font (size 1.27 1.27)) (justify left bottom))
   )
-  (label "A_IN_3" (at 154.94 241.935 180) (fields_autoplaced)
-    (effects (font (size 1.27 1.27)) (justify right bottom))
+  (label "A_IN_3_PIN" (at 226.06 178.435 0) (fields_autoplaced)
+    (effects (font (size 1.27 1.27)) (justify left bottom))
   )
   (label "QSPI_SD1" (at 80.01 146.685 0) (fields_autoplaced)
@@
     (effects (font (size 1.27 1.27)) (justify right))
   )
-  (hierarchical_label "A_IN_2" (shape output) (at 226.06 175.895 0) (fields_autoplaced)
-    (effects (font (size 1.27 1.27)) (justify left))
-  )
   (hierarchical_label "SCL1" (shape bidirectional) (at 226.06 173.355 0) (fields_autoplaced)
     (effects (font (size 1.27 1.27)) (justify left))
@@
     (effects (font (size 1.27 1.27)) (justify left))
   )
-  (hierarchical_label "A_IN_2" (shape input) (at 137.16 241.935 0) (fields_autoplaced)
-    (effects (font (size 1.27 1.27)) (justify left))
+  (hierarchical_label "A_IN_2" (shape input) (at 125.73 241.935 180) (fields_autoplaced)
+    (effects (font (size 1.27 1.27)) (justify right))
   )
   (hierarchical_label "ROT_ENC_1" (shape input) (at 226.06 165.735 0) (fields_autoplaced)
@@
     (effects (font (size 1.27 1.27)) (justify right))
   )
-  (hierarchical_label "A_IN_3" (shape output) (at 226.06 178.435 0) (fields_autoplaced)
-    (effects (font (size 1.27 1.27)) (justify left))
-  )
   (hierarchical_label "TFT_CS" (shape output) (at 245.11 125.095 0) (fields_autoplaced)
     (effects (font (size 1.27 1.27)) (justify left))
@@
     (effects (font (size 1.27 1.27)) (justify left))
   )
-  (hierarchical_label "A_IN_3" (shape input) (at 166.37 241.935 0) (fields_autoplaced)
-    (effects (font (size 1.27 1.27)) (justify left))
+  (hierarchical_label "A_IN_3" (shape input) (at 157.48 241.935 180) (fields_autoplaced)
+    (effects (font (size 1.27 1.27)) (justify right))
   )
   (hierarchical_label "CAN_H" (shape bidirectional) (at 384.81 106.68 0) (fields_autoplaced)
@@
     )
   )
-  (symbol (lib_id "2.passive:R") (at 160.02 241.935 90) (unit 1)
+  (symbol (lib_id "2.passive:R") (at 162.56 241.935 90) (unit 1)
     (in_bom yes) (on_board yes) (dnp no)
-    (property "Reference" "R28" (at 158.115 240.03 90)
+    (property "Reference" "R28" (at 160.655 240.03 90)
       (effects (font (size 1.27 1.27)) (justify right))
     )
-    (property "Value" "10k" (at 158.115 238.125 90)
+    (property "Value" "10k" (at 160.655 238.125 90)
       (effects (font (size 1.27 1.27)) (justify right))
     )
-    (property "Footprint" "2_Passives_Resistors_SMD_IPC:R_1608_603_B" (at 160.02 243.713 90)
-      (effects (font (size 1.27 1.27)) hide)
-    )
-    (property "Datasheet" "~" (at 160.02 241.935 0)
+    (property "Footprint" "2_Passives_Resistors_SMD_IPC:R_1608_603_B" (at 162.56 243.713 90)
+      (effects (font (size 1.27 1.27)) hide)
+    )
+    (property "Datasheet" "~" (at 162.56 241.935 0)
       (effects (font (size 1.27 1.27)) hide)
     )
@@
     )
   )
-  (symbol (lib_id "0.power-symbols:GND") (at 165.1 251.46 0) (unit 1)
-    (in_bom yes) (on_board yes) (dnp no) (fields_autoplaced)
-    (property "Reference" "#PWR099" (at 165.1 257.81 0)
-      (effects (font (size 1.27 1.27)) hide)
-    )
-    (property "Value" "GND" (at 165.1 255.5955 0)
-      (effects (font (size 1.27 1.27)))
-    )
-    (property "Footprint" "" (at 165.1 251.46 0)
-      (effects (font (size 1.27 1.27)) hide)
-    )
-    (property "Datasheet" "" (at 165.1 251.46 0)
+  (symbol (lib_id "0.power-symbols:GND") (at 167.64 251.46 0) (unit 1)
+    (in_bom yes) (on_board yes) (dnp no) (fields_autoplaced)
+    (property "Reference" "#PWR099" (at 167.64 257.81 0)
+      (effects (font (size 1.27 1.27)) hide)
+    )
+    (property "Value" "GND" (at 167.64 255.5955 0)
+      (effects (font (size 1.27 1.27)))
+    )
+    (property "Footprint" "" (at 167.64 251.46 0)
+      (effects (font (size 1.27 1.27)) hide)
+    )
+    (property "Datasheet" "" (at 167.64 251.46 0)
       (effects (font (size 1.27 1.27)) hide)
     )
@@
     )
   )
-  (symbol (lib_id "1.semi.discrete:D_Zener") (at 165.1 247.015 270) (unit 1)
+  (symbol (lib_id "1.semi.discrete:D_Zener") (at 167.64 247.015 270) (unit 1)
     (in_bom yes) (on_board yes) (dnp no)
-    (property "Reference" "D9" (at 155.575 246.364 90)
-      (effects (font (size 1.27 1.27)) (justify left))
-    )
-    (property "Value" "D_Zener" (at 155.575 248.285 90)
-      (effects (font (size 1.27 1.27)) (justify left))
-    )
-    (property "Footprint" "project_footprints:SOD-323" (at 165.1 247.015 0)
-      (effects (font (size 1.27 1.27)) hide)
-    )
-    (property "Datasheet" "~" (at 165.1 247.015 0)
-      (effects (font (size 1.27 1.27)) hide)
-    )
+    (property "Reference" "D9" (at 158.115 246.364 90)
+      (effects (font (size 1.27 1.27)) (justify left))
+    )
+    (property "Value" "D_Zener" (at 158.115 248.285 90)
+      (effects (font (size 1.27 1.27)) (justify left))
+    )
+    (property "Footprint" "project_footprints:SOD-323" (at 167.64 247.015 0)
+      (effects (font (size 1.27 1.27)) hide)
+    )
+    (property "Datasheet" "~" (at 167.64 247.015 0)
+      (effects (font (size 1.27 1.27)) hide)
+    )

Commit message: preliminary finish
Parts:
- removed D6: WS2812B, 1_Semi_LED-Opto:WS2812B, symbol 1.semi.opto:WS2812B
- added C33: 1uF, 2_Passives_Resistors_SMD_IPC:R_1005_402_A, symbol 2.passive:C
- added NT1: net-tie, 0_NetTie:NetTie-2_SMD_Pad0.5mm, symbol 0.power-symbols:net-tie
Connections:
- net +3V3: now also C33.1
- net GND: now also C33.2, NT1.2; no longer C10.2, C11.2, C12.2, C13.2, C14.2, C15.2, C16.2, C17.2, C25.2, C4.1, C5.2, C7.2, C8.2, C9.2, U10.19 (TESTEN), U10.57 (GND), Y3.2, Y3.4
- net LED_CTL: no longer names the net of U10.9 (GPIO7)
- new net GNDD: C10.2, C11.2, C12.2, C13.2, C14.2, C15.2, C16.2, C17.2, C25.2, C4.1, C5.2, C7.2, C8.2, C9.2, NT1.1, U10.19 (TESTEN), U10.57 (GND), Y3.2, Y3.4
Other:
- moved on the sheet: C23, C24, D1
