File: eOPRA_interface/processor.kicad_sch (KiCad schematic)
At the start: 46 parts, among them SW1 SW_Push, U10 RP2040, U11 W25Q128JVS, U13 MCP25625, Y1 16Mhz 12pF, Y3 12Mhz 12pF

Commit message: draft 2 wifi finish
Connections:
- net ESP_INT: now reaches U10.9 (GPIO7)
- no-connect marks 5 -> 4
Changed lines of the file:
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@@
   (no_connect (at 310.515 149.225))
   (no_connect (at 339.725 149.225))
-  (no_connect (at 226.06 120.015))
   (no_connect (at 339.725 102.87))
   (no_connect (at 310.515 151.765))
@@
   (hierarchical_label "~{RESET}" (shape input) (at 158.115 102.235 180) (fields_autoplaced)
     (effects (font (size 1.27 1.27)) (justify right))
+  )
+  (hierarchical_label "ESP_INT" (shape output) (at 226.06 120.015 0) (fields_autoplaced)
+    (effects (font (size 1.27 1.27)) (justify left))
   )
   (hierarchical_label "TFT_DC" (shape output) (at 226.06 114.935 0) (fields_autoplaced)
@@
     )
   )
+  (symbol (lib_id "2.passive:C") (at 358.14 111.76 0) (unit 1)
+    (in_bom yes) (on_board yes) (dnp no) (fields_autoplaced)
+    (property "Reference" "C33" (at 361.061 111.1163 0)
+      (effects (font (size 1.27 1.27)) (justify left))
+    )
+    (property "Value" "1uF" (at 361.061 113.0373 0)
+      (effects (font (size 1.27 1.27)) (justify left))
+    )
+    (property "Footprint" "2_Passives_Resistors_SMD_IPC:R_1005_402_A" (at 359.1052 115.57 0)
+      (effects (font (size 1.27 1.27)) hide)
+    )
+    (property "Datasheet" "~" (at 358.14 111.76 0)
+      (effects (font (size 1.27 1.27)) hide)
+    )
+    (pin "1")
+    (pin "2")
+    (instances
+      (project "eOPRA_interface"
+        (path "/9f7a57db-2daa-452d-a1aa-74a4ad8115df/d165d604-1acf-4179-9574-6e327e7130e7"
+          (reference "C33") (unit 1)
+        )
+      )
+    )
+  )
   (symbol (lib_id "2.passive:R") (at 36.83 244.475 0) (unit 1)
     (in_bom yes) (on_board yes) (dnp no)
@@
         )
       )
-    )
-  )
-  (symbol (lib_id "2.passive:C") (at 358.14 111.76 0) (unit 1)
-    (in_bom yes) (on_board yes) (dnp no) (fields_autoplaced)
-    (property "Reference" "C33" (at 361.061 111.1163 0)
-      (effects (font (size 1.27 1.27)) (justify left))
-    )
-    (property "Value" "1uF" (at 361.061 113.0373 0)
-      (effects (font (size 1.27 1.27)) (justify left))
-    )
-    (property "Footprint" "2_Passives_Resistors_SMD_IPC:R_1005_402_A" (at 359.1052 115.57 0)
-      (effects (font (size 1.27 1.27)) hide)
-    )
-    (property "Datasheet" "~" (at 358.14 111.76 0)
-      (effects (font (size 1.27 1.27)) hide)
-    )
-    (pin "1")
-    (pin "2")
-    (instances
-      (project "eOPRA_interface"
-        (path "/9f7a57db-2daa-452d-a1aa-74a4ad8115df/d165d604-1acf-4179-9574-6e327e7130e7"
-          (reference "C33") (unit 1)
-        )
-      )

Commit message: stuff
Parts:
- removed R16: 500, 2_Passives_Resistors_SMD_IPC:R_1608_603_B, symbol 2.passive:R
- added JP4: ~, 0_misc:SolderJumper-2_P1.3mm_Bridged_RoundedPad1.0x1.5mm, symbol 2.passive:Jumper_NC_Small
- added R13, R14: 27k4, 2_Passives_Resistors_SMD_IPC:R_1005_402_A, symbol 2.passive:R
- added R49: 10k, 2_Passives_Resistors_SMD_IPC:R_1608_603_B, symbol 2.passive:R
- added R80: 120, 2_Passives_Resistors_SMD_IPC:R_1005_402_A, symbol 2.passive:R
- C10, C11, C12, C13, C14, C15, C25, C7, C8, C9: value 100nF -> 0.1uF; PN (none) -> 2,1
- C10: value 0.1u -> 0.1uF; footprint 2_Passives_Capacitors_SMD_IPC:C_1608_603_B -> 2_Passives_Capacitors_SMD_IPC:C_1005_402_A; PN (none) -> 2,1
- C16, C17, C21, C22, C33, C4, C5: footprint 2_Passives_Resistors_SMD_IPC:R_1005_402_A -> 2_Passives_Capacitors_SMD_IPC:C_1005_402_A; PN (none) -> 2,2
- C23, C24: footprint 2_Passives_Resistors_SMD_IPC:R_1005_402_A -> 2_Passives_Capacitors_SMD_IPC:C_1005_402_A; PN (none) -> 2,5
- D1: footprint 1_Semi_TO_SOT:SOT-23 -> 1_Semi_TO_SOT:SOT-323_SC-70; PN (none) -> 3,1
- D3: PN (none) -> 3,3
- D8, D9: PN (none) -> 3,4
- R11, R15, R25, R27, R28: PN (none) -> 1,2
- R17, R4: PN (none) -> 1,3
- R81: footprint 2_Passives_Resistors_SMD_IPC:R_1005_402_A -> 2_Passives_Resistors_SMD_IPC:R_1608_603_B; PN (none) -> 1,4
- R97: PN (none) -> 1,6
- SW1: PN (none) -> 9,4
- TP3: value TEST -> ~
- U10: PN (none) -> 4,3
- U11: value W25Q128JVS -> W25Q128JVP; PN (none) -> 4,4
- U13: PN (none) -> 4,5
- Y1: PN Q 16,0-JXS32-12-10/15-T1-WA-LF -> 7,2
- Y3: PN RH100-12.000-12-1010-X-TR-NS2 -> 7,1
Connections:
- net +3V3: now also R49.2
- net A_IN_2_PIN: now also U10.38 (GPIO26_ADC0); no longer U10.40 (GPIO28_ADC2)
- net A_IN_3_PIN: now also U10.39 (GPIO27_ADC1); no longer U10.41 (GPIO29_ADC3)
- net CAN_CS: now also U10.40 (GPIO28_ADC2); no longer U10.30 (GPIO19)
- net CAN_H: now also R80.2
- net CAN_L: now also JP4.1
- net CAN_RESET: now also U10.41 (GPIO29_ADC3); no longer U10.29 (GPIO18)
- net QSPI_CS: now also R49.1
- net SCL1: now also U10.30 (GPIO19); no longer U10.39 (GPIO27_ADC1)
- net SDA1: now also U10.29 (GPIO18); no longer U10.38 (GPIO26_ADC0)
- net USB_D+: now also R13.1; no longer U10.47 (USB_D+)
- net USB_D-: now also R14.1; no longer U10.46 (USB_D-)
- net GNDD renamed GNDISO1
- new net: R14.2, U10.46 (USB_D-)
- new net: JP4.2, R80.1
- new net: R13.2, U10.47 (USB_D+)
Other:
- note added: "Place termination resistors close to RP2040"
- moved on the sheet: C23, C24, D1, D8, D9, NT1, R27, R28
