File: eOPRA_interface/switch_control.kicad_sch (KiCad schematic)
At the start: 11 parts, among them Q1 G3VM-351VY1-TR05, Q7 G3VM-351VY1-TR05, Q7 Q_NMOS_GSD, U4 74HC154

Commit message: schematic v1.0 finished
Parts:
- removed Q7: Q_NMOS_GSD, 1_Semi_TO_SOT:SOT-323FL, symbol 1.semi.discrete:Q_NMOS_GSD
- removed R16: 300, 2_Passives_Resistors_SMD_IPC:R_1608_603_B, symbol 2.passive:R
- removed R31: R, symbol 2.passive:R
- removed R49: 10k, 2_Passives_Resistors_SMD_IPC:R_1608_603_B, symbol 2.passive:R
- removed U4: 74HC154, symbol 1.semi.ic.logic:74HC154
- added D3: LED, 1_Semi_Discrete_Diodes_SMD:D_0603, symbol 1.semi.opto:LED
- added Q11, Q14, Q15, Q17, Q18, Q20, Q22, Q23, Q26, Q27, Q30, Q31, Q34, Q9: G3VM-351VY1-TR05, project_footprints:G3VM-351VY1-TR05, symbol 1.semi.discrete:Q_MOS_SS_Relay
- added Q7 (x15): Q_NMOS_GSD, 1_Semi_TO_SOT:SOT-323FL, symbol 1.semi.discrete:Q_NMOS_GSD
- added R16 (x15): 300, 2_Passives_Resistors_SMD_IPC:R_1608_603_B, symbol 2.passive:R
- added R32, R35, R38, R4, R43, R44, R48, R49, R55, R56, R61, R62, R67, R68, R73, R74: 500, 2_Passives_Resistors_SMD_IPC:R_1608_603_B, symbol 2.passive:R
- added R49 (x15): 10k, 2_Passives_Resistors_SMD_IPC:R_1608_603_B, symbol 2.passive:R
- added SW4: SW_SPST, project_footprints:AS11AH, symbol 3.electromechanical.switch:SW_SPST
- added U17: 74HC238, project_footprints:QFN50P250X350X100-17N, symbol 1.semi.ic.logic.74xx_IEEE:74HC238
- Q1, Q7: footprint (none) -> project_footprints:G3VM-351VY1-TR05
- Q7: PN 4,11 -> (none)
- R16: PN 1,10 -> (none)
- R49: PN 1,5 -> (none)
- R5: value R -> 500; footprint (none) -> 2_Passives_Resistors_SMD_IPC:R_1608_603_B
Connections:
- net +3V3: now also Q11.1, Q14.1, Q15.1, Q17.1, Q18.1, Q20.1, Q22.1, Q23.1, Q26.1, Q27.1, Q30.1, Q31.1, Q34.1, Q9.1, R4.1, U17.16, U17.4 (~{G2A}), U17.5 (~{G2B})
- net ECN_CTL_0: now also U17.1 (A0)
- net ECN_CTL_1: now also U17.2 (A1)
- net ECN_CTL_2: now also U17.3 (A2)
- net EMG_HIGH: now also Q14.4, Q15.4, Q20.4, Q23.4, Q26.4, Q31.4, Q9.4
- net EMG_LOW: now also Q11.4, Q17.4, Q18.4, Q22.4, Q27.4, Q30.4, Q34.4
- net GND: now also Q7.2 (S), Q7.2 (S), Q7.2 (S), Q7.2 (S), Q7.2 (S), Q7.2 (S), Q7.2 (S), Q7.2 (S), Q7.2 (S), Q7.2 (S), Q7.2 (S), Q7.2 (S), Q7.2 (S), Q7.2 (S), Q7.2 (S), R49.1, R49.1, R49.1, R49.1, R49.1, R49.1, R49.1, R49.1, R49.1, R49.1, R49.1, R49.1, R49.1, R49.1, R49.1, SW4.2 (B), U17.8 (GND)
- net at Q7.2: now also R32.2
- net CHAN_1a renamed CHAN_0
- net CHAN_0: now also R16.2, R49.2, U17.15 (Y0)
- net CHAN_1a_OUT renamed CHAN_0A_OUT
- net CHAN_1b_OUT renamed CHAN_0B_OUT
- new net: Q20.2, R55.2
- new net: Q7.1 (G), R16.1 (x15)
- new net: Q7.3 (D), R49.1
- new net: Q18.2, R49.2
- new net: D3.1 (K), SW4.1 (A), U17.6 (G1)
- new net: D3.2 (A), R4.2
- new net: Q7.3 (D), R73.1
- new net: Q31.2, R68.2
- new net: Q7.3 (D), R48.1
- new net: Q34.2, R74.2
- new net: Q7.3 (D), R44.1
- new net: Q22.2, R61.2
- new net: Q7.3 (D), R56.1
- new net: Q7.3 (D), R68.1
- new net: Q17.2, R48.2
- new net: Q7.3 (D), R43.1
- new net: Q15.2, R44.2
- new net: Q11.2, R38.2
- new net: Q7.3 (D), R61.1
- new net: Q26.2, R67.2
- new net: Q7.3 (D), R38.1
- new net: Q7.3 (D), R67.1
- new net: Q14.2, R43.2
- new net: Q7.3 (D), R35.1
- new net: Q9.2, R35.2
- new net: Q7.3 (D), R62.1
- new net: Q27.2, R62.2
- new net: Q7.3 (D), R74.1
- new net: Q7.3 (D), R32.1
- new net: Q23.2, R56.2
- new net: Q30.2, R73.2
- new net: Q7.3 (D), R55.1
- new net CHAN_1: R16.2, R16.2, R49.2, R49.2, U17.14 (Y1)
- new net CHAN_1A_OUT: Q14.3
- new net CHAN_1B_OUT: Q17.3
- new net CHAN_2: R16.2, R16.2, R49.2, R49.2, U17.13 (Y2)
- new net CHAN_2A_OUT: Q9.3
- new net CHAN_2B_OUT: Q11.3
- new net CHAN_3: R16.2, R16.2, R49.2, R49.2, U17.12 (Y3)
- new net CHAN_3A_OUT: Q15.3
- new net CHAN_3B_OUT: Q18.3
- new net CHAN_4: R16.2, R16.2, R49.2, R49.2, U17.11 (Y4)
- new net CHAN_4A_OUT: Q20.3
- new net CHAN_4B_OUT: Q22.3
- new net CHAN_5: R16.2, R16.2, R49.2, R49.2, U17.10 (Y5)
- new net CHAN_5A_OUT: Q26.3
- new net CHAN_5B_OUT: Q30.3
- new net CHAN_6: R16.2, R16.2, R49.2, R49.2, U17.9 (Y6)
- new net CHAN_6A_OUT: Q23.3
- new net CHAN_6B_OUT: Q27.3
- new net CHAN_7: R16.2, R16.2, R49.2, R49.2, U17.7 (Y7)
- new net CHAN_7A_OUT: Q31.3
- new net CHAN_7B_OUT: Q34.3
- no-connect marks 2 -> 0
Other:
- note added: "CHANNEL 0"
- note added: "CHANNEL 1"
- note added: "CHANNEL 2"
- note added: "CHANNEL 3"
- note added: "CHANNEL 4"
- note added: "CHANNEL 5"
- note added: "CHANNEL 6"
- note added: "CHANNEL 7"
- moved on the sheet: Q1, Q7, R16, R49, R5

Commit message: Version updates
Other:
- company: (none) -> Massachusetts Institute of Technology / MIT Media Lab
- title: (none) -> eOPRA Switch / Stimulation Controller
Changed lines of the file:
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@@
 (kicad_sch (version 20230121) (generator eeschema)
   (paper "A3")
+  (title_block
+    (title "eOPRA Switch / Stimulation Controller")
+    (date "2023-08-01")
+    (rev "1.0")
+    (company "Massachusetts Institute of Technology / MIT Media Lab")
+  )
   (junction (at 52.07 233.68) (diameter 0) (color 0 0 0 0)
   )

Commit message: before esp
Connections:
- net GND: no longer Q7.2 (S), Q7.2 (S), Q7.2 (S), Q7.2 (S), Q7.2 (S), Q7.2 (S), Q7.2 (S), Q7.2 (S), Q7.2 (S), Q7.2 (S), Q7.2 (S), Q7.2 (S), Q7.2 (S), Q7.2 (S), Q7.2 (S), Q7.2 (S), R49.1, R49.1, R49.1, R49.1, R49.1, R49.1, R49.1, R49.1, R49.1, R49.1, R49.1, R49.1, R49.1, R49.1, R49.1, R49.1
- net +3V3 renamed SWITCHING_3V3
- new net GNDD: Q7.2 (S), Q7.2 (S), Q7.2 (S), Q7.2 (S), Q7.2 (S), Q7.2 (S), Q7.2 (S), Q7.2 (S), Q7.2 (S), Q7.2 (S), Q7.2 (S), Q7.2 (S), Q7.2 (S), Q7.2 (S), Q7.2 (S), Q7.2 (S), R49.1, R49.1, R49.1, R49.1, R49.1, R49.1, R49.1, R49.1, R49.1, R49.1, R49.1, R49.1, R49.1, R49.1, R49.1, R49.1
Other:
- moved on the sheet: D3, R4, SW4, U17

Commit message: preliminary finish
Connections:
- net GNDD is gone; now on net GNDREF: Q7.2 (S), Q7.2 (S), Q7.2 (S), Q7.2 (S), Q7.2 (S), Q7.2 (S), Q7.2 (S), Q7.2 (S), Q7.2 (S), Q7.2 (S), Q7.2 (S), Q7.2 (S), Q7.2 (S), Q7.2 (S), Q7.2 (S), Q7.2 (S), R49.1, R49.1, R49.1, R49.1, R49.1, R49.1, R49.1, R49.1, R49.1, R49.1, R49.1, R49.1, R49.1, R49.1, R49.1, R49.1
- net GND renamed GNDREF

Commit message: stuff
Parts:
- added TP5 (x24): ~, 0_misc:test_point_0.8mm_square, symbol 5.connector.interconnect:TEST
- D3: PN (none) -> 3,3
- Q1, Q11, Q14, Q15, Q17, Q18, Q20, Q22, Q23, Q26, Q27, Q30, Q31, Q34, Q7, Q9: PN (none) -> 9,1
- Q7: PN (none) -> 10,1
- R16: PN (none) -> 1,5
- R32, R35, R38, R4, R43, R44, R48, R49, R5, R55, R56, R61, R62, R67, R68, R73, R74: PN (none) -> 1,4
- R49: PN (none) -> 1,2
- SW4: PN (none) -> 9,5
- U17: value 74HC238 -> ~; PN (none) -> 4,7
Connections:
- net CHAN_0: now also TP5.1
- net CHAN_0A_OUT: now also TP5.1
- net CHAN_0B_OUT: now also TP5.1
- net CHAN_1: now also TP5.1
- net CHAN_1A_OUT: now also TP5.1
- net CHAN_1B_OUT: now also TP5.1
- net CHAN_2: now also TP5.1
- net CHAN_2A_OUT: now also TP5.1
- net CHAN_2B_OUT: now also TP5.1
- net CHAN_3: now also TP5.1
- net CHAN_3A_OUT: now also TP5.1
- net CHAN_3B_OUT: now also TP5.1
- net CHAN_4: now also TP5.1
- net CHAN_4A_OUT: now also TP5.1
- net CHAN_4B_OUT: now also TP5.1
- net CHAN_5: now also TP5.1
- net CHAN_5A_OUT: now also TP5.1
- net CHAN_5B_OUT: now also TP5.1
- net CHAN_6: now also TP5.1
- net CHAN_6A_OUT: now also TP5.1
- net CHAN_6B_OUT: now also TP5.1
- net CHAN_7: now also TP5.1
- net CHAN_7A_OUT: now also TP5.1
- net CHAN_7B_OUT: now also TP5.1
- net GNDREF: now also U17.4 (~{G2A}), U17.5 (~{G2B})
- net SWITCHING_3V3: no longer U17.4 (~{G2A}), U17.5 (~{G2B})
- net at D3.1 (K), SW4.1 (A): no longer U17.6 (G1)
- net at D3.2 (A), R4.2: now also U17.6 (G1)
Other:
- moved on the sheet: D3, R4, SW4, U17

Commit message: stuff
Parts:
- removed R4: 500, 2_Passives_Resistors_SMD_IPC:R_1608_603_B, symbol 2.passive:R
- added R17: 300, 2_Passives_Resistors_SMD_IPC:R_1608_603_B, symbol 2.passive:R
- added R49 (x3): N/A, 2_Passives_Resistors_SMD_IPC:R_1608_603_B, symbol 2.passive:R
- Q7: value Q_NMOS_GSD -> RU1J002YNTCL
- R32, R35, R38, R43, R44, R48, R49, R5, R55, R56, R61, R62, R67, R68, R73, R74: value 500 -> 300; PN 1,4 -> 1,5
- SW4: value SW_SPST -> ~
Connections:
- net CHAN_5A_OUT: now also R49.2
- net CHAN_5B_OUT: now also R49.1
- net CHAN_6A_OUT: now also R49.2
- net CHAN_6B_OUT: now also R49.1
- net CHAN_7A_OUT: now also R49.2
- net CHAN_7B_OUT: now also R49.1
- net GNDREF: now also D3.1 (K); no longer SW4.2 (B)
- net SWITCHING_3V3: now also SW4.2 (B)
- net at SW4.1 (A): now also U17.6 (G1), R17.2; no longer D3.1 (K)
- net at D3.2 (A): now also R17.1; no longer U17.6 (G1)
Other:
- note added: "Channel load resistors (Optional)"
- note added: "Decoder"
- note added: "refer to: https://www.digitimer.com/wp-content/uploads/2020/07/Digitimer-Application-Note_DS5-and-D188_v2.pdf"
- moved on the sheet: D3, TP5, U17
