File: eOPRA_interface/regulator.kicad_sch (KiCad schematic)
At the start: 10 parts, among them U14 AP2205-50, U34 AP2213-8_SOIC

Commit message: schematic v1.0 finished
Parts:
- removed C33: 1u, 2_Passives_Capacitors_SMD_IPC:C_1608_603_B, symbol 2.passive:C
- removed C34: 100p, 2_Passives_Capacitors_SMD_IPC:C_1608_603_B, symbol 2.passive:C
- removed C80: 10u, 2_Passives_Capacitors_SMD_IPC:C_2012_805_B, symbol 2.passive:C
- removed U34: AP2213-8_SOIC, 1_Semi_Misc:SOIC-8_3.9x4.9mm_P1.27mm, symbol 1.semi.ic.pmic.voltagereg:AP2213-8_SOIC
- added C11, C15: 10u, 2_Passives_Capacitors_SMD_IPC:C_2012_805_B, symbol 2.passive:C
- added R29: 75k, 2_Passives_Resistors_SMD_IPC:R_1608_603_B, symbol 2.passive:R
- added R32: 102k, 2_Passives_Resistors_SMD_IPC:R_1608_603_B, symbol 2.passive:R
- added R33: 32.4k, 2_Passives_Resistors_SMD_IPC:R_1608_603_B, symbol 2.passive:R
- added U4: MPM3610, 1_Semi_QFN:20-PowerLQFN, symbol 1.semi.ic.pmic.voltagereg:MPM3610
- D1, D2: PN TBD -> (none)
Connections:
- net +3V3: now also C15.2, R32.1, U4.9 (OUT)
- net GND: now also C11.2, C15.1, R33.2, U4.12 (PGND), U4.13 (PGND), U4.14 (PGND), U4.3 (AGND)
- net SYS_PWR: now also C11.1, R29.1, U4.16 (IN)
- net BATT_1_PWR renamed +BATT
- new net: R32.2, R33.1, U4.1 (FB)
- new net: R29.2, U4.17 (EN)
- no-connect marks 0 -> 4
Other:
- note added: "Vin = 2.3V-24V Vout = 5V @150mA"
- note removed: "Vin = 2.3V-24V Vout = 3.3V @150mA"
- note removed: "Vin = 2.5V-18V Vout = 3.3V @500mA"
- moved on the sheet: C33, D1, D2, U14

Commit message: Version updates
Other:
- company: (none) -> Massachusetts Institute of Technology / MIT Media Lab
- title: (none) -> eOPRA Switch / Stimulation Controller
Changed lines of the file:
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@@
 (kicad_sch (version 20230121) (generator eeschema)
   (paper "A4")
+  (title_block
+    (title "eOPRA Switch / Stimulation Controller")
+    (date "2023-08-01")
+    (rev "1.0")
+    (company "Massachusetts Institute of Technology / MIT Media Lab")
+  )
   (junction (at 125.095 86.36) (diameter 0) (color 0 0 0 0)
   )

Commit message: before esp
Parts:
- removed C11, C15: 10u, 2_Passives_Capacitors_SMD_IPC:C_2012_805_B, symbol 2.passive:C
- removed C33: 1u, 2_Passives_Capacitors_SMD_IPC:C_1608_603_B, symbol 2.passive:C
- removed R29: 75k, 2_Passives_Resistors_SMD_IPC:R_1608_603_B, symbol 2.passive:R
- removed R32: 102k, 2_Passives_Resistors_SMD_IPC:R_1608_603_B, symbol 2.passive:R
- removed R33: 32.4k, 2_Passives_Resistors_SMD_IPC:R_1608_603_B, symbol 2.passive:R
- removed U4: MPM3610, 1_Semi_QFN:20-PowerLQFN, symbol 1.semi.ic.pmic.voltagereg:MPM3610
- added C33 (x2): 1u, 2_Passives_Capacitors_SMD_IPC:C_1608_603_B, symbol 2.passive:C
- added C34 (x2): 100p, 2_Passives_Capacitors_SMD_IPC:C_1608_603_B, symbol 2.passive:C
- added C80 (x3): 10u, 2_Passives_Capacitors_SMD_IPC:C_2012_805_B, symbol 2.passive:C
- added U34 (x2): AP2213-8_SOIC, 1_Semi_Misc:SOIC-8_3.9x4.9mm_P1.27mm, symbol 1.semi.ic.pmic.voltagereg:AP2213-8_SOIC
Connections:
- net +3V3: now also C80.2, U34.3 (VOUT)
- net +5V: now also C80.2
- net GND: now also C33.1, C33.1, C34.2, C80.1, C80.1, U34.5 (GND), U34.5 (GND), U34.6 (GND), U34.6 (GND), U34.7 (GND), U34.8 (GND)
- net SYS_PWR: now also C33.2, C33.2, U34.1 (EN), U34.1 (EN), U34.2 (VIN), U34.2 (VIN)
- new net: C34.1, U34.4 (BYP) (x2)
- new net GNDD: C34.2, C80.1, U34.7 (GND), U34.8 (GND)
- new net SWITCHING_3V3: C80.2, U34.3 (VOUT)
- no-connect marks 4 -> 0
Other:
- note added: "Vin = 2.5V-18V Vout = 3.3V @500mA"
- moved on the sheet: C33, D1, D2, U14

Commit message: preliminary finish
Parts:
- added NT1: net-tie, 0_NetTie:NetTie-2_SMD_Pad0.5mm, symbol 0.power-symbols:net-tie
Connections:
- net GNDD is gone; now on net GND: C34.2, C80.1, U34.7 (GND), U34.8 (GND)
- net GND: now also NT1.2
- new net GNDREF: NT1.1
Changed lines of the file:
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@@
+    (stroke (width 0) (type default))
+  )
+  (wire (pts (xy 187.325 126.365) (xy 187.325 121.92))
     (stroke (width 0) (type default))
   )
@@
     (stroke (width 0) (type default))
   )
+  (wire (pts (xy 187.325 121.92) (xy 186.055 121.92))
+    (stroke (width 0) (type default))
+  )
   (wire (pts (xy 190.5 87.63) (xy 184.15 87.63))
     (stroke (width 0) (type default))
@@
     (stroke (width 0) (type default))
   )
+  (wire (pts (xy 180.34 121.92) (xy 180.975 121.92))
+    (stroke (width 0) (type default))
+  )
   (wire (pts (xy 60.325 76.2) (xy 62.23 76.2))
     (stroke (width 0) (type default))
   )
+  (wire (pts (xy 171.45 123.19) (xy 171.45 126.365))
+    (stroke (width 0) (type default))
+  )
   (wire (pts (xy 213.995 78.74) (xy 208.915 78.74))
     (stroke (width 0) (type default))
@@
     (stroke (width 0) (type default))
   )
+  (wire (pts (xy 180.34 126.365) (xy 180.34 121.92))
+    (stroke (width 0) (type default))
+  )
   (wire (pts (xy 140.335 118.11) (xy 140.97 118.11))
     (stroke (width 0) (type default))
@@
     (stroke (width 0) (type default))
   )
-  (wire (pts (xy 151.765 124.46) (xy 151.765 125.73))
+  (wire (pts (xy 151.765 124.46) (xy 151.765 126.365))
     (stroke (width 0) (type default))
   )
@@
     (property "Intersheetrefs" "${INTERSHEET_REFS}" (at 151.765 93.7049 90)
       (effects (font (size 1.27 1.27)) (justify left) hide)
+    )
+  )
+  (symbol (lib_id "0.power-symbols:GNDREF") (at 180.34 126.365 0) (unit 1)
+    (in_bom yes) (on_board yes) (dnp no) (fields_autoplaced)
+    (property "Reference" "#PWR065" (at 180.34 132.715 0)
+      (effects (font (size 1.27 1.27)) hide)
+    )
+    (property "Value" "GNDREF" (at 180.34 130.4981 0)
+      (effects (font (size 1.27 1.27)))
+    )
+    (property "Footprint" "" (at 180.34 126.365 0)
+      (effects (font (size 1.27 1.27)) hide)
+    )
+    (property "Datasheet" "" (at 180.34 126.365 0)
+      (effects (font (size 1.27 1.27)) hide)
+    )
+    (pin "1")
+    (instances
+      (project "eOPRA_interface"
+        (path "/9f7a57db-2daa-452d-a1aa-74a4ad8115df/70fa3f7a-75da-4226-ac71-3f9e913064ed"
+          (reference "#PWR065") (unit 1)
+        )
+        (path "/9f7a57db-2daa-452d-a1aa-74a4ad8115df/16a508a1-14d6-439d-afb0-bad239c786d4"
+          (reference "#PWR080") (unit 1)
+        )
+      )
     )
   )
@@
     )
   )
+  (symbol (lib_id "0.power-symbols:PWR_FLAG") (at 171.45 123.19 0) (unit 1)
+    (in_bom yes) (on_board yes) (dnp no) (fields_autoplaced)
+    (property "Reference" "#FLG04" (at 171.45 121.285 0)
+      (effects (font (size 1.27 1.27)) hide)
+    )
+    (property "Value" "PWR_FLAG" (at 171.45 119.0569 0)
+      (effects (font (size 1.27 1.27)))
+    )
+    (property "Footprint" "" (at 171.45 123.19 0)
+      (effects (font (size 1.27 1.27)) hide)
+    )
+    (property "Datasheet" "" (at 171.45 123.19 0)
+      (effects (font (size 1.27 1.27)) hide)
+    )
+    (pin "1")
+    (instances
+      (project "eOPRA_interface"
+        (path "/9f7a57db-2daa-452d-a1aa-74a4ad8115df/16a508a1-14d6-439d-afb0-bad239c786d4"
+          (reference "#FLG04") (unit 1)
+        )
+      )
+    )
+  )
   (symbol (lib_id "0.power-symbols:GND") (at 88.9 85.725 0) (unit 1)
     (in_bom yes) (on_board yes) (dnp no) (fields_autoplaced)
@@
         (path "/9f7a57db-2daa-452d-a1aa-74a4ad8115df/16a508a1-14d6-439d-afb0-bad239c786d4"
           (reference "#PWR08") (unit 1)
+        )
+      )
+    )
+  )
+  (symbol (lib_id "0.power-symbols:GNDREF") (at 171.45 126.365 0) (unit 1)
+    (in_bom yes) (on_board yes) (dnp no) (fields_autoplaced)
+    (property "Reference" "#PWR065" (at 171.45 132.715 0)
+      (effects (font (size 1.27 1.27)) hide)
+    )
+    (property "Value" "GNDREF" (at 171.45 130.4981 0)
+      (effects (font (size 1.27 1.27)))
+    )
+    (property "Footprint" "" (at 171.45 126.365 0)
+      (effects (font (size 1.27 1.27)) hide)
+    )
+    (property "Datasheet" "" (at 171.45 126.365 0)
+      (effects (font (size 1.27 1.27)) hide)
+    )
+    (pin "1")
+    (instances
+      (project "eOPRA_interface"
+        (path "/9f7a57db-2daa-452d-a1aa-74a4ad8115df/70fa3f7a-75da-4226-ac71-3f9e913064ed"
+          (reference "#PWR065") (unit 1)
+        )
+        (path "/9f7a57db-2daa-452d-a1aa-74a4ad8115df/16a508a1-14d6-439d-afb0-bad239c786d4"
+          (reference "#PWR079") (unit 1)
         )
       )
@@
     )
   )
-  (symbol (lib_id "0.power-symbols:GNDD") (at 151.765 125.73 0) (unit 1)
-    (in_bom yes) (on_board yes) (dnp no) (fields_autoplaced)
-    (property "Reference" "#PWR096" (at 151.765 132.08 0)
-      (effects (font (size 1.27 1.27)) hide)
-    )
-    (property "Value" "GNDD" (at 151.765 129.8655 0)
-      (effects (font (size 1.27 1.27)))
-    )
-    (property "Footprint" "" (at 151.765 125.73 0)
-      (effects (font (size 1.27 1.27)) hide)
-    )
-    (property "Datasheet" "" (at 151.765 125.73 0)
-      (effects (font (size 1.27 1.27)) hide)
-    )
-    (pin "1")
-    (instances
-      (project "eOPRA_interface"
-        (path "/9f7a57db-2daa-452d-a1aa-74a4ad8115df/16a508a1-14d6-439d-afb0-bad239c786d4"
-          (reference "#PWR096") (unit 1)
+  (symbol (lib_id "0.power-symbols:net-tie") (at 183.515 120.65 0) (unit 1)
+    (in_bom yes) (on_board yes) (dnp no)
+    (property "Reference" "NT1" (at 183.515 117.0974 0)
+      (effects (font (size 0.7874 0.7874)))
+    )
+    (property "Value" "net-tie" (at 183.515 118.745 0)
+      (effects (font (size 0.7874 0.7874)))
+    )
+    (property "Footprint" "0_NetTie:NetTie-2_SMD_Pad0.5mm" (at 183.515 120.65 0)
+      (effects (font (size 0.7874 0.7874)) hide)
+    )
+    (property "Datasheet" "" (at 183.515 120.65 0)
+      (effects (font (size 0.7874 0.7874)) hide)
+    )
+    (pin "1")
+    (pin "2")
+    (instances
+      (project "eOPRA_interface"
+        (path "/9f7a57db-2daa-452d-a1aa-74a4ad8115df/d165d604-1acf-4179-9574-6e327e7130e7"
+          (reference "NT1") (unit 1)
+        )
+        (path "/9f7a57db-2daa-452d-a1aa-74a4ad8115df/16a508a1-14d6-439d-afb0-bad239c786d4"
+          (reference "NT2") (unit 1)
+        )
+      )
+    )
+  )
+  (symbol (lib_id "0.power-symbols:GND") (at 187.325 126.365 0) (unit 1)
+    (in_bom yes) (on_board yes) (dnp no) (fields_autoplaced)
+    (property "Reference" "#PWR081" (at 187.325 132.715 0)
+      (effects (font (size 1.27 1.27)) hide)
+    )
+    (property "Value" "GND" (at 187.325 130.4981 0)
+      (effects (font (size 1.27 1.27)))
+    )
+    (property "Footprint" "" (at 187.325 126.365 0)
+      (effects (font (size 1.27 1.27)) hide)
+    )
+    (property "Datasheet" "" (at 187.325 126.365 0)
+      (effects (font (size 1.27 1.27)) hide)
+    )
+    (pin "1")
+    (instances
+      (project "eOPRA_interface"
+        (path "/9f7a57db-2daa-452d-a1aa-74a4ad8115df/16a508a1-14d6-439d-afb0-bad239c786d4"
+          (reference "#PWR081") (unit 1)
         )
       )
@@
     )
   )
-  (symbol (lib_id "0.power-symbols:GND") (at 115.57 125.73 0) (unit 1)
-    (in_bom yes) (on_board yes) (dnp no) (fields_autoplaced)
-    (property "Reference" "#PWR042" (at 115.57 132.08 0)
-      (effects (font (size 1.27 1.27)) hide)
-    )
-    (property "Value" "GND" (at 115.57 129.8655 0)
-      (effects (font (size 1.27 1.27)))
-    )
-    (property "Footprint" "" (at 115.57 125.73 0)
-      (effects (font (size 1.27 1.27)) hide)
-    )
-    (property "Datasheet" "" (at 115.57 125.73 0)
-      (effects (font (size 1.27 1.27)) hide)
-    )
-    (pin "1")
-    (instances
-      (project "eOPRA_interface"
-        (path "/9f7a57db-2daa-452d-a1aa-74a4ad8115df/16a508a1-14d6-439d-afb0-bad239c786d4"
-          (reference "#PWR042") (unit 1)
-        )
-      )
-    )
-  )
   (symbol (lib_id "2.passive:C") (at 184.15 80.645 180) (unit 1)
     (in_bom yes) (on_board yes) (dnp no)
@@
     )
   )
+  (symbol (lib_id "0.power-symbols:GND") (at 151.765 126.365 0) (unit 1)
+    (in_bom yes) (on_board yes) (dnp no) (fields_autoplaced)
+    (property "Reference" "#PWR042" (at 151.765 132.715 0)
+      (effects (font (size 1.27 1.27)) hide)
+    )
+    (property "Value" "GND" (at 151.765 130.4981 0)
+      (effects (font (size 1.27 1.27)))
+    )
+    (property "Footprint" "" (at 151.765 126.365 0)
+      (effects (font (size 1.27 1.27)) hide)
+    )
+    (property "Datasheet" "" (at 151.765 126.365 0)
+      (effects (font (size 1.27 1.27)) hide)
+    )
+    (pin "1")
+    (instances
+      (project "eOPRA_interface"
+        (path "/9f7a57db-2daa-452d-a1aa-74a4ad8115df/16a508a1-14d6-439d-afb0-bad239c786d4"
+          (reference "#PWR042") (unit 1)
+        )
+      )
+    )
+  )
   (symbol (lib_id "0.power-symbols:+3.3V") (at 220.345 74.295 0) (unit 1)
     (in_bom yes) (on_board yes) (dnp no) (fields_autoplaced)
@@
         )
       )
+    )
+  )
+  (symbol (lib_id "0.power-symbols:GND") (at 115.57 125.73 0) (unit 1)
+    (in_bom yes) (on_board yes) (dnp no) (fields_autoplaced)
+    (property "Reference" "#PWR09" (at 115.57 132.08 0)
+      (effects (font (size 1.27 1.27)) hide)
+    )
+    (property "Value" "GND" (at 115.57 129.8631 0)
+      (effects (font (size 1.27 1.27)))
+    )
+    (property "Footprint" "" (at 115.57 125.73 0)
+      (effects (font (size 1.27 1.27)) hide)
+    )
+    (property "Datasheet" "" (at 115.57 125.73 0)
+      (effects (font (size 1.27 1.27)) hide)
+    )
+    (pin "1")
+    (instances
+      (project "eOPRA_interface"
+        (path "/9f7a57db-2daa-452d-a1aa-74a4ad8115df/16a508a1-14d6-439d-afb0-bad239c786d4"
+          (reference "#PWR09") (unit 1)
+        )
+      )

Commit message: stuff
Parts:
- removed C80 (x3): 10u, 2_Passives_Capacitors_SMD_IPC:C_2012_805_B, symbol 2.passive:C
- added C16 (x3): 1uF, 2_Passives_Capacitors_SMD_IPC:C_1005_402_A, symbol 2.passive:C
- C33: value 1u -> 1uF; footprint 2_Passives_Capacitors_SMD_IPC:C_1608_603_B -> 2_Passives_Capacitors_SMD_IPC:C_1005_402_A; PN (none) -> 2,2
- C33: value 1u -> 1uF; footprint 2_Passives_Capacitors_SMD_IPC:C_1608_603_B -> 2_Passives_Capacitors_SMD_IPC:C_1005_402_A; PN 2,4 -> 2,2
- C34: PN STOCK -> 2,3; Part GCG1885G1H101JA01D -> (none)
- D1, D2: PN (none) -> 3,2; Part PMEG1030EH -> (none)
- U14: PN (none) -> 4,6
- U34: PN 4,10 -> 4,1
Connections:
- net +3V3: now also C16.1
- net +5V: now also C16.1
- net GND: now also C16.2, C16.2, C16.2
- net SWITCHING_3V3: now also C16.1

Commit message: stuff
Parts:
- C34: value 100p -> 100pF
Connections:
- net GND: no longer C16.2, C33.1
- new net GNDISO2: C16.2, C33.1
Changed lines of the file:
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@@
     (stroke (width 0) (type default))
   )
-  (wire (pts (xy 88.9 84.455) (xy 88.9 85.725))
+  (wire (pts (xy 88.9 84.455) (xy 88.9 86.36))
     (stroke (width 0) (type default))
   )
@@
     )
   )
-  (symbol (lib_id "0.power-symbols:GND") (at 88.9 85.725 0) (unit 1)
-    (in_bom yes) (on_board yes) (dnp no) (fields_autoplaced)
-    (property "Reference" "#PWR08" (at 88.9 92.075 0)
-      (effects (font (size 1.27 1.27)) hide)
-    )
-    (property "Value" "GND" (at 88.9 89.8605 0)
-      (effects (font (size 1.27 1.27)))
-    )
-    (property "Footprint" "" (at 88.9 85.725 0)
-      (effects (font (size 1.27 1.27)) hide)
-    )
-    (property "Datasheet" "" (at 88.9 85.725 0)
+  (symbol (lib_id "0.power-symbols:GND") (at 88.9 86.36 0) (unit 1)
+    (in_bom yes) (on_board yes) (dnp no) (fields_autoplaced)
+    (property "Reference" "#PWR08" (at 88.9 92.71 0)
+      (effects (font (size 1.27 1.27)) hide)
+    )
+    (property "Value" "GND" (at 88.9 90.4955 0)
+      (effects (font (size 1.27 1.27)))
+    )
+    (property "Footprint" "" (at 88.9 86.36 0)
+      (effects (font (size 1.27 1.27)) hide)
+    )
+    (property "Datasheet" "" (at 88.9 86.36 0)
       (effects (font (size 1.27 1.27)) hide)
     )
@@
     )
   )
-  (symbol (lib_id "0.power-symbols:GND") (at 125.095 86.36 0) (unit 1)
-    (in_bom yes) (on_board yes) (dnp no) (fields_autoplaced)
-    (property "Reference" "#PWR046" (at 125.095 92.71 0)
-      (effects (font (size 1.27 1.27)) hide)
-    )
-    (property "Value" "GND" (at 125.095 90.4955 0)
-      (effects (font (size 1.27 1.27)))
-    )
-    (property "Footprint" "" (at 125.095 86.36 0)
-      (effects (font (size 1.27 1.27)) hide)
-    )
-    (property "Datasheet" "" (at 125.095 86.36 0)
-      (effects (font (size 1.27 1.27)) hide)
-    )
-    (pin "1")
-    (instances
-      (project "eOPRA_interface"
-        (path "/9f7a57db-2daa-452d-a1aa-74a4ad8115df/16a508a1-14d6-439d-afb0-bad239c786d4"
-          (reference "#PWR046") (unit 1)
-        )
-      )
-    )
-  )
   (symbol (lib_id "1.semi.discrete:D_Schottky") (at 53.34 76.2 180) (unit 1)
     (in_bom yes) (on_board yes) (dnp no)
@@
       (effects (font (size 1.27 1.27)) (justify left))
     )
-    (property "Value" "100p" (at 143.51 126.365 0)
+    (property "Value" "100pF" (at 143.51 126.365 0)
       (effects (font (size 1.27 1.27)) (justify left))
     )
@@
     )
   )
+  (symbol (lib_id "0.power-symbols:GNDISO2") (at 125.095 86.36 0) (unit 1)
+    (in_bom yes) (on_board yes) (dnp no) (fields_autoplaced)
+    (property "Reference" "#PWR051" (at 125.095 92.71 0)
+      (effects (font (size 1.27 1.27)) hide)
+    )
+    (property "Value" "GNDISO2" (at 125.095 90.4931 0)
+      (effects (font (size 1.27 1.27)))
+    )
+    (property "Footprint" "" (at 125.095 86.36 0)
+      (effects (font (size 1.27 1.27)) hide)
+    )
+    (property "Datasheet" "" (at 125.095 86.36 0)
+      (effects (font (size 1.27 1.27)) hide)
+    )
+    (pin "1")
+    (instances
+      (project "eOPRA_interface"
+        (path "/9f7a57db-2daa-452d-a1aa-74a4ad8115df/d165d604-1acf-4179-9574-6e327e7130e7"
+          (reference "#PWR051") (unit 1)
+        )
+        (path "/9f7a57db-2daa-452d-a1aa-74a4ad8115df/16a508a1-14d6-439d-afb0-bad239c786d4"
+          (reference "#PWR046") (unit 1)
+        )
+      )
+    )
+  )
   (symbol (lib_id "2.passive:C") (at 184.15 80.645 180) (unit 1)
     (in_bom yes) (on_board yes) (dnp no)
@@
       (effects (font (size 1.27 1.27)) (justify left))
     )
-    (property "Value" "100p" (at 212.09 89.535 0)
-      (effects (font (size 1.27 1.27)) (justify left))
-    )
+    (property "Value" "100pF" (at 212.09 89.535 0)
+      (effects (font (size 1.27 1.27)) (justify left))
+    )

Commit message: stuffs
Parts:
- added D3 (x3): LED, 1_Semi_Discrete_Diodes_SMD:D_0603, symbol 1.semi.opto:LED
- added R17 (x3): 300, 2_Passives_Resistors_SMD_IPC:R_1608_603_B, symbol 2.passive:R
Connections:
- net +3V3: now also R17.2
- net +5V: now also R17.2
- net GND: now also D3.1 (K), D3.1 (K)
- net GNDISO2: now also D3.1 (K)
- net SWITCHING_3V3: now also R17.2
- new net: D3.2 (A), R17.1 (x3)
