File: eOPRA_interface/eOPRA_interface.kicad_pcb (KiCad board)
At the start: 4 copper layers, 93.3 x 65 mm, 181 parts, among them J1 CONN_01X04_MALE, J2 CONN_01X04_MALE, J3 CONN_01X04_MALE, J4 CONN_01X02_MALE, J5 CONN_01X04_MALE, J6 CONN_02X10, J8 CONN_01X04_MALE, Q1 G3VM-351VY1-TR05, Q10 Q_NMOS_GSD, Q11 G3VM-351VY1-TR05, Q12 Q_NMOS_GSD, Q13 Q_NMOS_GSD, Q14 G3VM-351VY1-TR05, Q15 G3VM-351VY1-TR05, Q16 Q_NMOS_GSD, Q17 G3VM-351VY1-TR05, Q18 G3VM-351VY1-TR05, Q19 Q_NMOS_GSD, Q2 Q_NMOS_GSD, Q20 G3VM-351VY1-TR05, Q21 Q_NMOS_GSD, Q22 G3VM-351VY1-TR05, Q23 G3VM-351VY1-TR05, Q24 Q_NMOS_GSD, Q25 Q_NMOS_GSD, Q26 G3VM-351VY1-TR05, Q27 G3VM-351VY1-TR05, Q28 Q_NMOS_GSD, Q29 Q_NMOS_GSD, Q3 Q_NMOS_GSD, Q30 G3VM-351VY1-TR05, Q31 G3VM-351VY1-TR05, Q32 Q_NMOS_GSD, Q33 Q_NMOS_GSD, Q34 G3VM-351VY1-TR05, Q4 Q_NMOS_GSD, Q5 Q_PMOS_GSD, Q6 Q_NMOS_GSD, Q7 G3VM-351VY1-TR05, Q8 Q_NMOS_GSD, Q9 G3VM-351VY1-TR05, SW2 SW_Push, SW3 SW_Push, SW4 SW_SPST, SW6 SW_Push, SW7 Rotary_Encoder_Switch, U1 USB_C_2.0, U10 RP2040, U11 W25Q128JVS, U13 MCP25625, U14 AP2205-50, U16 MPM3610, U17 74HC238, U2 ARM-SWD-10, U4 DS3231MZ+, U5 XT-X, U6 Mounting-holes, U7 Mounting-holes, U8 Mounting-holes, U9 Mounting-holes, Y1 16Mhz 12pF, Y3 12Mhz 12pF

Commit message: before esp
Parts:
- removed R20: 75k, 2_Passives_Resistors_SMD_IPC:R_1608_603_B
- removed R23: 102k, 2_Passives_Resistors_SMD_IPC:R_1608_603_B
- removed R80: 32.4k, 2_Passives_Resistors_SMD_IPC:R_1608_603_B
- removed TP1: TEST, 0_misc:test_point_2mm_square
- removed U16: MPM3610, 1_Semi_QFN:20-PowerLQFN
- added C1: 1u, 2_Passives_Capacitors_SMD_IPC:C_1608_603_B, F.Cu at (166.3, 92.1)
- added C2: 100p, 2_Passives_Capacitors_SMD_IPC:C_1608_603_B, F.Cu at (162.1, 92.1)
- added C3: 10u, 2_Passives_Capacitors_SMD_IPC:C_2012_805_B, F.Cu at (167.0, 89.0)
- added C30: 10u, 2_Passives_Capacitors_SMD_IPC:C_2012_805_B, F.Cu at (203.4, 82.6)
- added U15: AP2213-8_SOIC, 1_Semi_Misc:SOIC-8_3.9x4.9mm_P1.27mm, F.Cu at (198.8, 84.4)
- added U3: AP2213-8_SOIC, 1_Semi_Misc:SOIC-8_3.9x4.9mm_P1.27mm, F.Cu at (162.3, 88.6)
- C20: value 1u -> 10u; footprint 2_Passives_Capacitors_SMD_IPC:C_1608_603_B -> 2_Passives_Capacitors_SMD_IPC:C_2012_805_B
- C28: value 10u -> 1u; footprint 2_Passives_Capacitors_SMD_IPC:C_2012_805_B -> 2_Passives_Capacitors_SMD_IPC:C_1608_603_B
- C29: value 10u -> 100p; footprint 2_Passives_Capacitors_SMD_IPC:C_2012_805_B -> 2_Passives_Capacitors_SMD_IPC:C_1608_603_B
- F1, JP1, Q10, Q12, Q13, Q16, Q19, Q2, Q21, Q24, Q25, Q28, Q29, Q32, Q33, Q4, Q5, Q6, Q8, R19, R26, R3, R30, R31, R32, R33, R34, R35, R36, R37, R38, R39, R40, R41, R42, R43, R44, R45, R46, R47, R48, R49, R5, R50, R52, R53, R54, R55, R56, R57, R58, R59, R60, R61, R62, R63, R64, R65, R66, R67, R68, R69, R70, R71, R72, R73, R74, TP2: moved to B.Cu
- R17: value 500 -> 1k; footprint 2_Passives_Resistors_SMD_IPC:R_1608_603_B -> 2_Passives_Resistors_SMD_IPC:R_1005_402_A
- U5: moved to F.Cu
- moved Q14 187.8 mm to (222.1, 83.0), turned to -90 degrees
- moved Q15 185.2 mm to (218.1, 83.0), turned to -90 degrees
- moved Q1 183.0 mm to (222.1, 91.0), turned to -90 degrees
- moved Q7 182.2 mm to (222.1, 117.8), turned to 90 degrees
- moved Q9 180.3 mm to (218.1, 91.0), turned to -90 degrees
- moved Q11 178.2 mm to (218.1, 117.8), turned to 90 degrees
- moved Q17 173.2 mm to (222.1, 109.9), turned to 90 degrees
- moved Q26 172.9 mm to (214.1, 83.0), turned to -90 degrees
- moved Q18 169.2 mm to (218.0, 109.9), turned to 90 degrees
- moved Q20 167.6 mm to (214.2, 91.0), turned to -90 degrees
- moved Q23 165.6 mm to (210.2, 91.0), turned to -90 degrees
- moved Q22 165.2 mm to (214.0, 117.9), turned to 90 degrees
- moved Q2 161.1 mm to (221.3, 93.2), turned to 180 degrees
- moved Q12 160.7 mm to (221.4, 85.2), turned to 180 degrees
- moved R26 160.6 mm to (222.8, 90.3), turned to 90 degrees
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Connections:
- C28 pad 1: /regulator/SYS_PWR -> GND
- C28 pad 2: GND -> /regulator/SYS_PWR
- C29 pad 1: GND -> Net-(U15-BYP)
- C29 pad 2: +3V3 -> GNDD
- Q1 pad 1: +3V3 -> SWITCHING_3V3
- Q10 pad 2: GND -> GNDD
- Q11 pad 1: +3V3 -> SWITCHING_3V3
- Q12 pad 2: GND -> GNDD
- Q13 pad 2: GND -> GNDD
- Q14 pad 1: +3V3 -> SWITCHING_3V3
- Q15 pad 1: +3V3 -> SWITCHING_3V3
- Q16 pad 2: GND -> GNDD
- Q17 pad 1: +3V3 -> SWITCHING_3V3
- Q18 pad 1: +3V3 -> SWITCHING_3V3
- Q19 pad 2: GND -> GNDD
- Q2 pad 2: GND -> GNDD
- Q20 pad 1: +3V3 -> SWITCHING_3V3
- Q21 pad 2: GND -> GNDD
- Q22 pad 1: +3V3 -> SWITCHING_3V3
- Q23 pad 1: +3V3 -> SWITCHING_3V3
- Q24 pad 2: GND -> GNDD
- Q25 pad 2: GND -> GNDD
- Q26 pad 1: +3V3 -> SWITCHING_3V3
- Q27 pad 1: +3V3 -> SWITCHING_3V3
- Q28 pad 2: GND -> GNDD
- Q29 pad 2: GND -> GNDD
- Q30 pad 1: +3V3 -> SWITCHING_3V3
- Q31 pad 1: +3V3 -> SWITCHING_3V3
- Q32 pad 2: GND -> GNDD
- Q33 pad 2: GND -> GNDD
- Q34 pad 1: +3V3 -> SWITCHING_3V3
- Q4 pad 2: GND -> GNDD
- Q6 pad 2: GND -> GNDD
- Q7 pad 1: +3V3 -> SWITCHING_3V3
- Q8 pad 2: GND -> GNDD
- Q9 pad 1: +3V3 -> SWITCHING_3V3
- R13 pad 1: /USB_D+ -> Net-(R13-Pad1)
- R13 pad 2: Net-(U10-USB_DP) -> /USB_D-
- R14 pad 1: /USB_D- -> Net-(R14-Pad1)
- R14 pad 2: Net-(U10-USB_DM) -> /USB_D+
- R17 pad 1: Net-(D3-A) -> /processor/QSPI_CS
- R17 pad 2: /processor/QSPI_CS -> Net-(D3-A)
- R19 pad 1: GND -> GNDD
- R29 pad 1: +3V3 -> SWITCHING_3V3
- R3 pad 1: GND -> GNDD
- R30 pad 1: GND -> GNDD
- R33 pad 1: GND -> GNDD
- R36 pad 1: GND -> GNDD
- R39 pad 1: GND -> GNDD
- R40 pad 1: GND -> GNDD
- R45 pad 1: GND -> GNDD
- R50 pad 1: GND -> GNDD
- R52 pad 1: GND -> GNDD
- R57 pad 1: GND -> GNDD
- R58 pad 1: GND -> GNDD
- R63 pad 1: GND -> GNDD
- R64 pad 1: GND -> GNDD
- R69 pad 1: GND -> GNDD
- R70 pad 1: GND -> GNDD
- U1 pad A6: /USB_D+ -> Net-(R14-Pad1)
- U1 pad A7: /USB_D- -> Net-(R13-Pad1)
- U1 pad B6: /USB_D+ -> Net-(R14-Pad1)
- U1 pad B7: /USB_D- -> Net-(R13-Pad1)
- U10 pad 46: Net-(U10-USB_DM) -> /USB_D-
- U10 pad 47: Net-(U10-USB_DP) -> /USB_D+
- U17 pad 16: +3V3 -> SWITCHING_3V3
- U17 pad 4: +3V3 -> SWITCHING_3V3
- U17 pad 5: +3V3 -> SWITCHING_3V3
- U2 pad 9: Net-(U2-GNDDetect) -> unconnected-(U2-GNDDetect-Pad9)
Routing:
- net GNDD: track 0.00 -> 155.5 mm
- net SWITCHING_3V3: track 0.00 -> 87.6 mm, vias 0 -> 15
- net EMG_LOW: track 0.00 -> 41.3 mm, vias 0 -> 4
- net EMG_HIGH: track 0.00 -> 38.4 mm, vias 0 -> 4
- net /switch_control/CHAN_3: track 0.00 -> 18.4 mm
- net /switch_control/CHAN_2: track 0.00 -> 18.2 mm
- net /switch_control/CHAN_5: track 0.00 -> 17.8 mm
- net /switch_control/CHAN_4: track 0.00 -> 17.6 mm
- net /switch_control/CHAN_7: track 0.00 -> 17.1 mm
- net /switch_control/CHAN_6: track 0.00 -> 17.1 mm
- net CHAN_7A_OUT: track 0.00 -> 16.5 mm
- net /switch_control/CHAN_0: track 0.00 -> 16.1 mm
- net /switch_control/CHAN_1: track 0.00 -> 16.0 mm
- net CHAN_5A_OUT: track 0.00 -> 14.6 mm
- net CHAN_0B_OUT: track 0.00 -> 14.1 mm
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- removed copper zone on F.Cu, net GND
Other:
- board size 93.3 x 65 mm -> 76 x 57.9 mm

Commit message: before 4 layer
Parts:
- J1, J8: moved to B.Cu
- moved R9 93.5 mm to (126.7, 116.5), turned to 180 degrees
- moved R10 89.6 mm to (129.8, 116.5)
- moved R21 74.9 mm to (126.7, 117.9)
- moved R12 72.8 mm to (129.8, 117.9), turned to 0 degrees
- moved U11 65.7 mm to (124.4, 86.2), turned to 90 degrees
- moved J1 53.0 mm to (118.7, 122.2), turned to 180 degrees
- moved C18 53.0 mm to (149.9, 48.7)
- moved R16 53.0 mm to (146.1, 48.7)
- moved R17 53.0 mm to (145.7, 47.4)
- moved D3 50.7 mm to (149.9, 47.2), turned to 180 degrees
- moved C1 48.3 mm to (118.1, 89.0)
- moved U3 46.6 mm to (115.8, 85.6)
- moved C3 46.6 mm to (120.4, 87.6)
- moved U5 46.2 mm to (119.4, 71.2)
- moved R8 45.2 mm to (115.2, 89.0), turned to 180 degrees
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Connections:
- D8 pad 1: /A_IN_2 -> /processor/A_IN_2_PIN
- D9 pad 1: /A_IN_3 -> /processor/A_IN_3_PIN
- Q3 pad 2: GNDD -> GND
- R1 pad 1: GNDD -> GND
- R2 pad 2: GNDD -> GND
- R27 pad 2: /A_IN_2 -> /processor/A_IN_2_PIN
- R28 pad 2: /A_IN_3 -> /processor/A_IN_3_PIN
- R6 pad 1: GNDD -> GND
- U1 pad A1: GNDD -> GND
- U1 pad A12: GNDD -> GND
- U1 pad B1: GNDD -> GND
- U1 pad B12: GNDD -> GND
- U1 pad S1: GNDD -> GND
- U10 pad 40: /A_IN_2 -> /processor/A_IN_2_PIN
- U10 pad 41: /A_IN_3 -> /processor/A_IN_3_PIN
- U2 pad 3: GNDD -> GND
- U2 pad 5: GNDD -> GND
Routing:
- net /regulator/SYS_PWR: track 0.00 -> 52.7 mm, vias 0 -> 1
- net /peripherals/~{TFT_RESET}: track 0.00 -> 42.2 mm
- net GND: track 2.52 -> 42.0 mm, vias 0 -> 14
- net +3V3: track 1.44 -> 39.4 mm, vias 0 -> 1
- net SWITCHING_3V3: track 87.6 -> 106.0 mm, vias 15 -> 17
- net EMG_HIGH: track 38.4 -> 56.2 mm
- net /processor/QSPI_SD1: track 0.00 -> 15.9 mm
- net /processor/QSPI_CS: track 0.00 -> 15.8 mm
- net VUSB: track 0.00 -> 15.0 mm
- net /switch_control/CHAN_7: track 17.1 -> 30.8 mm, vias 0 -> 1
- net /processor/QSPI_SD2: track 0.00 -> 13.6 mm
- net /processor/QSPI_SD3: track 0.00 -> 13.0 mm
- net /processor/QSPI_SCLK: track 0.00 -> 11.0 mm
- net GNDD: track 155.5 -> 164.4 mm, vias 0 -> 5
- net /processor/QSPI_SD0: track 0.00 -> 8.69 mm
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- added copper zone on B.Cu, net GND

Commit message: preliminary finish
Parts:
- removed D6: WS2812B, 1_Semi_LED-Opto:WS2812B
- added C31: 10u, 2_Passives_Capacitors_SMD_IPC:C_2012_805_B, F.Cu at (105.6, 107.5)
- added C32: 0.1u, 2_Passives_Capacitors_SMD_IPC:C_1608_603_B, F.Cu at (135.8, 93.5)
- added C33: 1uF, 2_Passives_Resistors_SMD_IPC:R_1005_402_A, F.Cu at (120.8, 108.6)
- added NT1: net-tie, 0_NetTie:NetTie-2_SMD_Pad0.5mm, B.Cu at (119.0, 101.7)
- added NT2: net-tie, 0_NetTie:NetTie-2_SMD_Pad0.5mm, F.Cu at (154.6, 79.9)
- C26, C27, J3, R10, R12, R21, R51, R75, R76, R77, R78, R79, R8, R9: moved to B.Cu
- moved U8 164.4 mm to (265.8, 70.5)
- moved U7 92.8 mm to (251.6, 64.2)
- moved U6 92.2 mm to (103.1, 121.9)
- moved C18 60.9 mm to (106.3, 91.2)
- moved R16 59.6 mm to (114.4, 99.1)
- moved J3 58.4 mm to (119.8, 122.2)
- moved D9 55.1 mm to (114.3, 121.9), turned to -90 degrees
- moved SW4 54.4 mm to (171.0, 79.0), turned to 90 degrees
- moved R28 53.0 mm to (114.6, 118.6), turned to 90 degrees
- moved C20 51.7 mm to (105.6, 104.2), turned to -90 degrees
- moved C22 51.6 mm to (106.7, 110.3), turned to -90 degrees
- moved D8 50.9 mm to (118.3, 116.2), turned to -90 degrees
- moved R27 50.9 mm to (116.6, 116.5), turned to 90 degrees
- moved C21 47.2 mm to (108.3, 107.5), turned to 180 degrees
- moved U14 46.4 mm to (108.3, 104.7), turned to -90 degrees
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Connections:
- C10 pad 2: GND -> GNDD
- C11 pad 2: GND -> GNDD
- C12 pad 2: GND -> GNDD
- C13 pad 2: GND -> GNDD
- C14 pad 2: GND -> GNDD
- C15 pad 2: GND -> GNDD
- C16 pad 2: GND -> GNDD
- C17 pad 2: GND -> GNDD
- C25 pad 2: GND -> GNDD
- C29 pad 2: GNDD -> GND
- C30 pad 1: GNDD -> GND
- C4 pad 1: GND -> GNDD
- C5 pad 2: GND -> GNDD
- C7 pad 2: GND -> GNDD
- C8 pad 2: GND -> GNDD
- C9 pad 2: GND -> GNDD
- Q10 pad 2: GNDD -> GNDREF
- Q12 pad 2: GNDD -> GNDREF
- Q13 pad 2: GNDD -> GNDREF
- Q16 pad 2: GNDD -> GNDREF
- Q19 pad 2: GNDD -> GNDREF
- Q2 pad 2: GNDD -> GNDREF
- Q21 pad 2: GNDD -> GNDREF
- Q24 pad 2: GNDD -> GNDREF
- Q25 pad 2: GNDD -> GNDREF
- Q28 pad 2: GNDD -> GNDREF
- Q29 pad 2: GNDD -> GNDREF
- Q32 pad 2: GNDD -> GNDREF
- Q33 pad 2: GNDD -> GNDREF
- Q4 pad 2: GNDD -> GNDREF
- Q6 pad 2: GNDD -> GNDREF
- Q8 pad 2: GNDD -> GNDREF
- R19 pad 1: GNDD -> GNDREF
- R3 pad 1: GNDD -> GNDREF
- R30 pad 1: GNDD -> GNDREF
- R33 pad 1: GNDD -> GNDREF
- R36 pad 1: GNDD -> GNDREF
- R39 pad 1: GNDD -> GNDREF
- R40 pad 1: GNDD -> GNDREF
- R45 pad 1: GNDD -> GNDREF
- R50 pad 1: GNDD -> GNDREF
- R52 pad 1: GNDD -> GNDREF
- R57 pad 1: GNDD -> GNDREF
- R58 pad 1: GNDD -> GNDREF
- R63 pad 1: GNDD -> GNDREF
- R64 pad 1: GNDD -> GNDREF
- R69 pad 1: GNDD -> GNDREF
- R70 pad 1: GNDD -> GNDREF
- SW4 pad 2: GND -> GNDREF
- U10 pad 19: GND -> GNDD
- U10 pad 57: GND -> GNDD
- U10 pad 9: /processor/LED_CTL -> unconnected-(U10-GPIO7-Pad9)
- U15 pad 7: GNDD -> GND
- U15 pad 8: GNDD -> GND
- U17 pad 17: unconnected-(U17-EP-Pad17) -> (no net)
- U17 pad 8: GND -> GNDREF
- Y3 pad 2: GND -> GNDD
- Y3 pad 4: GND -> GNDD
Routing:
- net GNDREF: track 0.00 -> 182.2 mm, vias 0 -> 8
- net GNDD: track 164.4 -> 23.5 mm, vias 5 -> 10
- net /~{RESET}: track 4.50 -> 72.7 mm, vias 0 -> 4
- net GND: track 42.0 -> 108.5 mm, vias 14 -> 37
- net /processor/ENC_CTL_0: track 0.00 -> 54.9 mm, vias 0 -> 3
- net /processor/ENC_CTL_1: track 0.00 -> 54.2 mm, vias 0 -> 3
- net /processor/ENC_CTL_2: track 0.00 -> 54.1 mm, vias 0 -> 3
- net +3V3: track 39.4 -> 91.8 mm, vias 1 -> 27
- net /ROT_ENC_0: track 1.20 -> 48.2 mm, vias 0 -> 2
- net /SCL1: track 2.01 -> 47.5 mm, vias 0 -> 3
- net /SDA1: track 1.83 -> 46.2 mm, vias 0 -> 3
- net /ROT_ENC_1: track 1.36 -> 44.4 mm, vias 0 -> 2
- net /switch_control/CHAN_2: track 18.2 -> 54.8 mm, vias 0 -> 3
- net /switch_control/CHAN_1: track 16.0 -> 50.9 mm, vias 0 -> 3
- net /processor/CAN_INT: track 0.00 -> 34.0 mm, vias 0 -> 3
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- added copper zone on In1.Cu, net +3V3
- added copper zone on In2.Cu, net GND
- added copper zone on B.Cu, net GNDD
- added copper zone on In2.Cu, net GNDREF
- added copper zone on In1.Cu, net SWITCHING_3V3
- removed copper zone on B.Cu, net GND
Other:
- board size 76 x 57.9 mm -> 75 x 50 mm

Commit message: draft 2 wifi finish
Parts:
- added C34: 1uF, 2_Passives_Resistors_SMD_IPC:R_1005_402_A, F.Cu at (151.8, 108.6)
- added C35: 1uF, 2_Passives_Resistors_SMD_IPC:R_1005_402_A, B.Cu at (146.5, 112.1)
- added D2: LED, 1_Semi_Discrete_Diodes_SMD:D_0603, F.Cu at (152.7, 118.5)
- added J7: CONN_01X04_MALE, project_footprints:JST_SM04B-GHS-TB(LF)(SN)-, B.Cu at (142.4, 122.1)
- added R20: 500, 2_Passives_Resistors_SMD_IPC:R_1608_603_B, F.Cu at (152.7, 117.0)
- added R22: 10k, 2_Passives_Resistors_SMD_IPC:R_1608_603_B, B.Cu at (146.6, 114.6)
- added SW1: SW_Push, project_footprints:TL3365AF180QG, B.Cu at (140.6, 113.0)
- added SW5: SW_Push, project_footprints:TL3365AF180QG, B.Cu at (144.1, 113.0)
- added TP1: TEST, 0_misc:test_point_1.0mm_square, B.Cu at (149.8, 111.1)
- added TP10: TEST, 0_misc:test_point_1.0mm_square, B.Cu at (134.7, 119.1)
- added TP11: TEST, 0_misc:test_point_1.0mm_square, B.Cu at (143.3, 107.6)
- added TP12: TEST, 0_misc:test_point_1.0mm_square, B.Cu at (141.3, 107.6)
- added TP13: TEST, 0_misc:test_point_1.0mm_square, B.Cu at (149.8, 123.1)
- added TP4: TEST, 0_misc:test_point_1.0mm_square, B.Cu at (144.3, 118.1)
- added TP5: TEST, 0_misc:test_point_1.0mm_square, B.Cu at (137.3, 107.5)
- added TP6: TEST, 0_misc:test_point_1.0mm_square, B.Cu at (147.3, 107.6)
- added TP7: TEST, 0_misc:test_point_1.0mm_square, B.Cu at (139.3, 107.6)
- added TP8: TEST, 0_misc:test_point_1.0mm_square, B.Cu at (145.3, 107.6)
- added TP9: TEST, 0_misc:test_point_1.0mm_square, B.Cu at (149.8, 113.1)
- added U16: ~, project_footprints:ESP8266-12E_ESP-12E, F.Cu at (142.3, 116.1)
- moved U8 123.7 mm to (153.2, 121.9)
- moved U7 99.3 mm to (153.2, 77.8)
- moved C5 3.66 mm to (127.8, 104.5), turned to 0 degrees
- moved C30 3.65 mm to (148.2, 76.2), turned to 180 degrees
- moved NT2 3.40 mm to (151.2, 80.2)
- moved C29 3.38 mm to (150.8, 83.0), turned to 90 degrees
- moved R7 2.23 mm to (120.7, 117.2)
- moved Q3 2.20 mm to (118.6, 118.0)
- moved R6 2.15 mm to (118.8, 115.1)
- moved R27 2.13 mm to (114.6, 117.3)
- moved D8 2.13 mm to (116.3, 116.9)
- moved SP1 1.82 mm to (123.1, 112.3)
- moved U15 1.38 mm to (147.3, 80.8)
- moved R28 1.08 mm to (113.8, 119.4), turned to 180 degrees
- moved C33 0.89 mm to (120.3, 107.9), turned to 90 degrees
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Connections:
- U10 pad 9: unconnected-(U10-GPIO7-Pad9) -> /ESP-Wifi/ESP_INT
Routing:
- net /TX: track 4.01 -> 34.2 mm, vias 2 -> 3
- net /RX: track 2.74 -> 32.4 mm, vias 1 -> 2
- net /ESP-Wifi/ESP_INT: track 0.00 -> 28.1 mm, vias 0 -> 3
- net /SCL1: track 47.5 -> 69.3 mm, vias 3 -> 4
- net /ESP-Wifi/EN: track 0.00 -> 12.6 mm, vias 0 -> 1
- net /RXD: track 0.00 -> 9.92 mm, vias 0 -> 1
- net /TXD: track 0.00 -> 9.36 mm, vias 0 -> 1
- net /ESP-Wifi/GPIO0: track 0.00 -> 9.31 mm, vias 0 -> 1
- net unconnected-(U7-Pad1): track 0.00 -> 8.59 mm, vias 0 -> 1
- net SWITCHING_3V3: track 132.9 -> 124.7 mm, vias 13 -> 12
- net GND: track 108.5 -> 116.6 mm, vias 37 -> 46
- net /SDA1: track 46.2 -> 52.7 mm
- net +3V3: track 91.8 -> 97.6 mm, vias 27 -> 30
- net /A_IN_2: track 5.21 -> 8.75 mm
- net GNDREF: track 182.2 -> 185.7 mm
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
Commit message: stuff
Parts:
- removed C35: 1uF, 2_Passives_Resistors_SMD_IPC:R_1005_402_A
- added C36: 1uF, 2_Passives_Capacitors_SMD_IPC:C_1005_402_A, B.Cu at (165.7, 121.0)
- added D11: LED, 1_Semi_Discrete_Diodes_SMD:D_0603, F.Cu at (153.3, 115.8)
- added D12: LED, 1_Semi_Discrete_Diodes_SMD:D_0603, F.Cu at (153.2, 117.8)
- added D6: LED, 1_Semi_Discrete_Diodes_SMD:D_0603, B.Cu at (137.8, 111.1)
- added JP2: ~, 0_misc:SolderJumper-2_P1.3mm_Bridged_RoundedPad1.0x1.5mm, B.Cu at (135.2, 119.8)
- added JP3: ~, 0_misc:SolderJumper-2_P1.3mm_Bridged_RoundedPad1.0x1.5mm, B.Cu at (135.2, 117.2)
- added JP4: ~, 0_misc:SolderJumper-2_P1.3mm_Bridged_RoundedPad1.0x1.5mm, F.Cu at (119.8, 117.4)
- added Q35: Q_NMOS_GSD, 1_Semi_TO_SOT:SOT-323FL, B.Cu at (151.4, 116.1)
- added Q36: Q_NMOS_GSD, 1_Semi_TO_SOT:SOT-323FL, B.Cu at (151.4, 117.5)
- added R23: 27k4, 2_Passives_Resistors_SMD_IPC:R_1005_402_A, F.Cu at (127.2, 89.7)
- added R24: 27k4, 2_Passives_Resistors_SMD_IPC:R_1005_402_A, F.Cu at (128.2, 89.7)
- added R80: 120, 2_Passives_Resistors_SMD_IPC:R_1005_402_A, B.Cu at (119.8, 117.4)
- added R82: 10k, 2_Passives_Resistors_SMD_IPC:R_1608_603_B, B.Cu at (135.2, 111.0)
- added R83: 10k, 2_Passives_Resistors_SMD_IPC:R_1608_603_B, B.Cu at (145.5, 118.0)
- added R84: 10k, 2_Passives_Resistors_SMD_IPC:R_1608_603_B, B.Cu at (154.3, 114.7)
- added R85: 300, 2_Passives_Resistors_SMD_IPC:R_1608_603_B, B.Cu at (154.2, 116.1)
- added R86: 10k, 2_Passives_Resistors_SMD_IPC:R_1608_603_B, B.Cu at (154.3, 119.0)
- added R87: 300, 2_Passives_Resistors_SMD_IPC:R_1608_603_B, B.Cu at (154.3, 117.6)
- added TP14: ~, 0_misc:test_point_0.8mm_square, B.Cu at (158.5, 97.0)
- added TP15: ~, 0_misc:test_point_0.8mm_square, B.Cu at (164.1, 96.0)
- added TP16: ~, 0_misc:test_point_0.8mm_square, B.Cu at (157.5, 96.0)
- added TP17: ~, 0_misc:test_point_0.8mm_square, B.Cu at (157.5, 94.0)
- added TP18: ~, 0_misc:test_point_0.8mm_square, B.Cu at (164.1, 94.0)
- added TP19: ~, 0_misc:test_point_0.8mm_square, B.Cu at (158.5, 95.0)
- added TP20: ~, 0_misc:test_point_0.8mm_square, B.Cu at (163.1, 95.0)
- added TP21: ~, 0_misc:test_point_0.8mm_square, B.Cu at (163.1, 93.0)
- added TP22: ~, 0_misc:test_point_0.8mm_square, B.Cu at (158.5, 93.0)
- added TP23: ~, 0_misc:test_point_0.8mm_square, B.Cu at (164.1, 92.0)
- added TP24: ~, 0_misc:test_point_0.8mm_square, B.Cu at (157.5, 92.0)
- added TP25: ~, 0_misc:test_point_0.8mm_square, B.Cu at (157.5, 90.0)
- added TP26: ~, 0_misc:test_point_0.8mm_square, B.Cu at (164.1, 90.0)
- added TP27: ~, 0_misc:test_point_0.8mm_square, B.Cu at (158.5, 91.0)
- added TP28: ~, 0_misc:test_point_0.8mm_square, B.Cu at (163.1, 91.0)
- added TP29: ~, 0_misc:test_point_0.8mm_square, B.Cu at (141.0, 101.4)
- added TP3: TEST, 0_misc:test_point_1.0mm_square, B.Cu at (148.2, 117.1)
- added TP30: ~, 0_misc:test_point_0.8mm_square, B.Cu at (155.9, 104.3)
- added TP31: ~, 0_misc:test_point_0.8mm_square, B.Cu at (141.0, 93.1)
- added TP32: ~, 0_misc:test_point_0.8mm_square, B.Cu at (149.0, 93.0)
- added TP33: ~, 0_misc:test_point_0.8mm_square, B.Cu at (149.2, 89.1)
- added TP34: ~, 0_misc:test_point_0.8mm_square, B.Cu at (141.1, 88.9)
- added TP35: ~, 0_misc:test_point_0.8mm_square, B.Cu at (141.0, 84.8)
- added TP36: ~, 0_misc:test_point_0.8mm_square, B.Cu at (149.1, 84.9)
- C1, C19, C28, C6: value 1u -> 1uF; footprint 2_Passives_Capacitors_SMD_IPC:C_1608_603_B -> 2_Passives_Capacitors_SMD_IPC:C_1005_402_A
- C10, C11, C12, C13, C14, C15, C25, C7, C8, C9: value 100nF -> 0.1uF
- C16, C17, C21, C22, C23, C24, C33, C34, C4, C5: footprint 2_Passives_Resistors_SMD_IPC:R_1005_402_A -> 2_Passives_Capacitors_SMD_IPC:C_1005_402_A
- C18: value 0.1u -> 0.1uF; footprint 2_Passives_Capacitors_SMD_IPC:C_1608_603_B -> 2_Passives_Capacitors_SMD_IPC:C_1005_402_A
- C20, C3, C30: value 10u -> 1uF; footprint 2_Passives_Capacitors_SMD_IPC:C_2012_805_B -> 2_Passives_Capacitors_SMD_IPC:C_1005_402_A
- C26, C27: value 0.01u -> 0.1uF; footprint 2_Passives_Capacitors_SMD_IPC:C_1608_603_B -> 2_Passives_Capacitors_SMD_IPC:C_1005_402_A
- C31: value 10u -> 1uF; footprint 2_Passives_Capacitors_SMD_IPC:C_2012_805_B -> 2_Passives_Capacitors_SMD_IPC:C_1005_402_A; moved to B.Cu
- C32: value 0.1u -> 1uF; footprint 2_Passives_Capacitors_SMD_IPC:C_1608_603_B -> 2_Passives_Capacitors_SMD_IPC:C_1005_402_A
- D1: footprint 1_Semi_TO_SOT:SOT-23 -> 1_Semi_TO_SOT:SOT-323_SC-70
- D2: value LED -> D_Schottky; footprint 1_Semi_Discrete_Diodes_SMD:D_0603 -> 1_Semi_Discrete_Diodes_SMD:D_SOD-123F; moved to B.Cu
- D5, Q3, R6, R7: moved to B.Cu
- JP1: value Jumper -> ~; footprint 0_misc:SolderJumper-2_P1.3mm_Open_RoundedPad1.0x1.5mm -> 0_misc:SolderJumper-2_P1.3mm_Bridged_RoundedPad1.0x1.5mm
- Q5: footprint 1_Semi_TO_SOT:TO-252-2 -> project_footprints:SON_8DU-T1-GE3_VIS
- R13, R14: value 27.4 -> 10k; footprint 2_Passives_Resistors_SMD_IPC:R_1005_402_A -> 2_Passives_Resistors_SMD_IPC:R_1608_603_B; moved to B.Cu
- R16: value 500 -> 10k
- R20: value 500 -> 10k; moved to B.Cu
- R81: footprint 2_Passives_Resistors_SMD_IPC:R_1005_402_A -> 2_Passives_Resistors_SMD_IPC:R_1608_603_B
- TP10, TP4: footprint 0_misc:test_point_1.0mm_square -> 0_misc:test_point_0.8mm_square
- TP13: value TEST -> ~; footprint 0_misc:test_point_1.0mm_square -> 0_misc:test_point_0.8mm_square
- TP2: value TEST -> ~
- U11: value W25Q128JVS -> W25Q128JVP
- U17: value 74HC238 -> ~
- moved R13 53.3 mm to (166.9, 121.3), turned to 90 degrees
- moved TP10 47.0 mm to (158.3, 78.4)
- moved TP4 42.5 mm to (159.5, 78.4), turned to -90 degrees
- moved R14 30.9 mm to (137.9, 114.3)
- moved TP13 29.3 mm to (163.1, 97.0)
- moved C31 19.7 mm to (104.7, 87.8), turned to -90 degrees
- moved JP1 19.5 mm to (105.3, 108.7)
- moved R20 17.9 mm to (135.2, 113.1), turned to 180 degrees
- moved TP9 16.7 mm to (133.2, 115.1), turned to 180 degrees
- moved TP1 16.7 mm to (133.2, 113.1)
- moved Q3 14.8 mm to (131.4, 110.6)
- moved R7 13.8 mm to (130.6, 107.7), turned to 180 degrees
- moved R6 11.9 mm to (129.4, 109.8), turned to 90 degrees
- moved D2 5.10 mm to (148.2, 121.0), turned to 90 degrees
- moved D5 5.03 mm to (115.1, 82.1)
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Connections:
- net GNDD renamed GNDISO1
- C20 pad 1: GND -> +5V
- C20 pad 2: +5V -> GND
- C3 pad 1: GND -> +3V3
- C3 pad 2: +3V3 -> GND
- C30 pad 1: GND -> SWITCHING_3V3
- C30 pad 2: SWITCHING_3V3 -> GND
- D2 pad 1: GND -> +3V3
- J7 pad 1: Net-(J7-Pad1) -> Net-(D2-A)
- R13 pad 1: Net-(R13-Pad1) -> /peripherals/switch
- R13 pad 2: /USB_D- -> /ENC_BUTTON
- R14 pad 1: Net-(R14-Pad1) -> Net-(D6-K)
- R14 pad 2: /USB_D+ -> /ESP-Wifi/GPIO0
- R20 pad 1: /ESP-Wifi/LED_STATIC -> +3V3
- R20 pad 2: Net-(D2-A) -> /ESP-Wifi/GPIO2
- R22 pad 2: /ESP-Wifi/EN -> /ESP-Wifi/~{RESET}
- R79 pad 1: /ENC_BUTTON -> /peripherals/switch
- SW5 pad 1: /ESP-Wifi/EN -> /ESP-Wifi/~{RESET}
- SW5 pad 3: /ESP-Wifi/EN -> /ESP-Wifi/~{RESET}
- SW7 pad S1: /ENC_BUTTON -> /peripherals/switch
- TP1 pad 1: Net-(U16-IO13) -> /ESP-Wifi/GPIO2
- TP10 pad 1: Net-(U16-IO5) -> EMG_LOW
- TP13 pad 1: Net-(U16-RESET) -> CHAN_0A_OUT
- TP4 pad 1: Net-(J7-Pad1) -> EMG_HIGH
- TP9 pad 1: Net-(U16-IO12) -> /ESP-Wifi/GPIO0
- U1 pad A6: Net-(R14-Pad1) -> /USB_D+
- U1 pad A7: Net-(R13-Pad1) -> /USB_D-
- U1 pad B6: Net-(R14-Pad1) -> /USB_D+
- U1 pad B7: Net-(R13-Pad1) -> /USB_D-
- U10 pad 29: /processor/CAN_RESET -> /SDA1
- U10 pad 30: /processor/CAN_CS -> /SCL1
- U10 pad 38: /SDA1 -> /processor/A_IN_2_PIN
- U10 pad 39: /SCL1 -> /processor/A_IN_3_PIN
- U10 pad 40: /processor/A_IN_2_PIN -> /processor/CAN_CS
- U10 pad 41: /processor/A_IN_3_PIN -> /processor/CAN_RESET
- U10 pad 46: /USB_D- -> Net-(U10-USB_D-)
- U10 pad 47: /USB_D+ -> Net-(U10-USB_D+)
- U16 pad 1: Net-(U16-RESET) -> /ESP-Wifi/~{RESET}
- U16 pad 16: unconnected-(U16-IO15-Pad16) -> Net-(U16-IO15)
- U16 pad 17: /SDA1 -> /ESP-Wifi/GPIO2
- U16 pad 19: /ESP-Wifi/ESP_INT -> Net-(U16-IO4)
- U16 pad 4: /ESP-Wifi/LED_STATIC -> Net-(U16-IO16)
- U16 pad 5: /SCL1 -> /ESP-Wifi/ESP_INT
- U16 pad 6: Net-(U16-IO12) -> /ESP-Wifi/LED1
- U16 pad 7: Net-(U16-IO13) -> /ESP-Wifi/LED2
- U17 pad 4: SWITCHING_3V3 -> GNDREF
- U17 pad 5: SWITCHING_3V3 -> GNDREF
- U17 pad 6: Net-(D10-K) -> Net-(D10-A)
Routing:
- net /SCL1: track 69.3 -> 49.7 mm, vias 4 -> 2
- net SWITCHING_3V3: track 124.7 -> 142.2 mm
- net /ESP-Wifi/~{RESET}: track 0.00 -> 17.3 mm, vias 0 -> 1
- net /ESP-Wifi/ESP_INT: track 28.1 -> 44.6 mm, vias 3 -> 2
- net Net-(Q3-D): track 15.2 -> 2.08 mm
- net +3V3: track 97.6 -> 107.9 mm, vias 30 -> 34
- net /ESP-Wifi/LED1: track 0.00 -> 10.2 mm, vias 0 -> 1
- net /processor/CAN_RESET: track 26.6 -> 36.7 mm, vias 2 -> 3
- net /peripherals/~{TFT_RESET}: track 32.8 -> 41.5 mm, vias 0 -> 1
- net /ESP-Wifi/EN: track 12.6 -> 3.92 mm
- net unconnected-(U7-Pad1): track 8.59 -> 0.00 mm, vias 1 -> 0
- net /ESP-Wifi/LED2: track 0.00 -> 8.55 mm, vias 0 -> 1
- net /processor/CAN_CS: track 23.6 -> 31.9 mm, vias 2 -> 3
- net /TFT_CS: track 29.5 -> 21.6 mm
- net Net-(D10-K): track 11.0 -> 4.11 mm, vias 2 -> 0
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