File: eOPRA_interface/eOPRA_interface.kicad_pcb (KiCad board)
At the start: 4 copper layers, 75 x 50 mm, 247 parts, among them J1 CONN_01X04_MALE, J2 CONN_01X04_MALE, J3 CONN_01X04_MALE, J4 CONN_01X02_MALE, J5 CONN_01X04_MALE, J6 CONN_02X10, J7 CONN_01X04_MALE, J8 CONN_01X04_MALE, Q1 G3VM-351VY1-TR05, Q10 Q_NMOS_GSD, Q11 G3VM-351VY1-TR05, Q12 Q_NMOS_GSD, Q13 Q_NMOS_GSD, Q14 G3VM-351VY1-TR05, Q15 G3VM-351VY1-TR05, Q16 Q_NMOS_GSD, Q17 G3VM-351VY1-TR05, Q18 G3VM-351VY1-TR05, Q19 Q_NMOS_GSD, Q2 Q_NMOS_GSD, Q20 G3VM-351VY1-TR05, Q21 Q_NMOS_GSD, Q22 G3VM-351VY1-TR05, Q23 G3VM-351VY1-TR05, Q24 Q_NMOS_GSD, Q25 Q_NMOS_GSD, Q26 G3VM-351VY1-TR05, Q27 G3VM-351VY1-TR05, Q28 Q_NMOS_GSD, Q29 Q_NMOS_GSD, Q3 Q_NMOS_GSD, Q30 G3VM-351VY1-TR05, Q31 G3VM-351VY1-TR05, Q32 Q_NMOS_GSD, Q33 Q_NMOS_GSD, Q34 G3VM-351VY1-TR05, Q35 Q_NMOS_GSD, Q36 Q_NMOS_GSD, Q4 Q_NMOS_GSD, Q5 Q_PMOS_GSD, Q6 Q_NMOS_GSD, Q7 G3VM-351VY1-TR05, Q8 Q_NMOS_GSD, Q9 G3VM-351VY1-TR05, SW1 SW_Push, SW2 SW_Push, SW3 SW_Push, SW4 SW_SPST, SW5 SW_Push, SW6 SW_Push, SW7 Rotary_Encoder_Switch, U1 USB_C_2.0, U10 RP2040, U11 W25Q128JVP, U13 MCP25625, U14 AP2205-50, U15 AP2213-8_SOIC, U2 ARM-SWD-10, U3 AP2213-8_SOIC, U4 DS3231MZ+, U5 XT-X, U6 Mounting-holes, U7 Mounting-holes, U8 Mounting-holes, U9 Mounting-holes, Y1 16Mhz 12pF, Y3 12Mhz 12pF

Commit message: stuff
Parts:
- removed Q35, Q36: Q_NMOS_GSD, 1_Semi_TO_SOT:SOT-323FL
- added C35: 0.1uF, 2_Passives_Capacitors_SMD_IPC:C_1005_402_A, F.Cu at (118.3, 102.3)
- added G***: LOGO, project_ss:biomech, F.Cu at (136.5, 103.3)
- added G***: LOGO, project_ss:media_lab, B.Cu at (170.2, 122.1)
- added NT3: net-tie, 0_NetTie:NetTie-2_SMD_Pad0.5mm, B.Cu at (104.2, 107.0)
- added R88: N/A, 2_Passives_Resistors_SMD_IPC:R_1608_603_B, B.Cu at (160.8, 92.3)
- C2, C29: value 100p -> 100pF
- Q10, Q12, Q13, Q16, Q19, Q2, Q21, Q24, Q25, Q28, Q29, Q3, Q32, Q33, Q4, Q6, Q8: value Q_NMOS_GSD -> RU1J002YNTCL
- R11, R25, U14: moved to B.Cu
- R18: value 500 -> 1k; footprint 2_Passives_Resistors_SMD_IPC:R_1608_603_B -> 2_Passives_Resistors_SMD_IPC:R_1005_402_A
- R23, R24: value 27k4 -> 27.4
- R29, R32, R35, R38, R43, R44, R48, R49, R5, R55, R56, R61, R62, R67, R68, R73, R74: value 500 -> 300
- R81: footprint 2_Passives_Resistors_SMD_IPC:R_1608_603_B -> 2_Passives_Resistors_SMD_IPC:R_1005_402_A
- R84, R86: value 10k -> 120; footprint 2_Passives_Resistors_SMD_IPC:R_1608_603_B -> 2_Passives_Resistors_SMD_IPC:R_1005_402_A; moved to F.Cu
- R85, R87: value 300 -> N/A
- SW4: value SW_SPST -> ~
- moved R87 28.8 mm to (160.8, 89.5)
- moved R85 26.0 mm to (160.8, 90.9)
- moved J7 17.7 mm to (160.1, 122.1)
- moved NT1 16.4 mm to (132.8, 107.1), turned to -90 degrees
- moved D2 14.6 mm to (162.0, 116.5), turned to -90 degrees
- moved C36 12.0 mm to (171.2, 110.4)
- moved R13 11.4 mm to (170.0, 110.3)
- moved JP1 8.13 mm to (102.5, 116.3), turned to -90 degrees
- moved C33 8.01 mm to (116.8, 100.8), turned to 135 degrees
- moved R79 7.65 mm to (168.6, 110.3)
- moved C23 6.54 mm to (110.4, 100.3), turned to 135 degrees
- moved D1 6.46 mm to (108.5, 101.2), turned to -45 degrees
- moved C22 5.66 mm to (112.1, 111.8), turned to 45 degrees
- moved C24 5.50 mm to (107.6, 103.0), turned to 135 degrees
- moved R15 4.91 mm to (106.2, 104.7), turned to 135 degrees
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Connections:
- C19 pad 1: GND -> GNDISO2
- C20 pad 2: GND -> GNDISO2
- C21 pad 2: GND -> GNDISO2
- C22 pad 1: GND -> GNDISO2
- C23 pad 1: GND -> GNDISO2
- C24 pad 1: GND -> GNDISO2
- C33 pad 2: GND -> GNDISO2
- D1 pad 3: GND -> GNDISO2
- D10 pad 1: Net-(D10-K) -> GNDREF
- D11 pad 1: Net-(D11-K) -> GND
- D11 pad 2: +3V3 -> Net-(D11-A)
- D12 pad 1: Net-(D12-K) -> GND
- D12 pad 2: +3V3 -> Net-(D12-A)
- R15 pad 2: GND -> GNDISO2
- R29 pad 1: SWITCHING_3V3 -> Net-(D10-A)
- R29 pad 2: Net-(D10-A) -> Net-(SW4-A)
- R84 pad 1: GND -> Net-(D11-A)
- R85 pad 1: Net-(Q35-G) -> CHAN_6B_OUT
- R85 pad 2: /ESP-Wifi/LED2 -> CHAN_6A_OUT
- R86 pad 1: GND -> Net-(D12-A)
- R87 pad 1: Net-(Q36-G) -> CHAN_7B_OUT
- R87 pad 2: /ESP-Wifi/LED1 -> CHAN_7A_OUT
- SW4 pad 1: Net-(D10-K) -> Net-(SW4-A)
- SW4 pad 2: GNDREF -> SWITCHING_3V3
- U13 pad 18: GND -> GNDISO2
- U13 pad 22: GND -> GNDISO2
- U13 pad 29: GND -> GNDISO2
- U17 pad 6: Net-(D10-A) -> Net-(SW4-A)
- Y1 pad 2: GND -> GNDISO2
- Y1 pad 4: GND -> GNDISO2
Routing:
- net GND: track 117.7 -> 87.9 mm, vias 54 -> 44
- net +3V3: track 107.9 -> 85.6 mm, vias 34 -> 33
- net /TXD: track 9.36 -> 30.8 mm
- net /RXD: track 9.92 -> 30.6 mm
- net GNDISO2: track 0.00 -> 16.3 mm, vias 0 -> 12
- net /processor/MISO1: track 26.5 -> 12.3 mm
- net Net-(SW4-A): track 0.00 -> 10.8 mm, vias 0 -> 2
- net /processor/MOSI1: track 25.0 -> 14.5 mm
- net /processor/CAN_CS: track 31.9 -> 42.2 mm, vias 3 -> 5
- net /processor/CAN_INT: track 34.5 -> 25.8 mm, vias 3 -> 2
- net /processor/~{Tx0RTS}: track 16.6 -> 25.0 mm
- net /processor/CAN_RESET: track 36.7 -> 44.2 mm, vias 3 -> 5
- net /peripherals/switch: track 4.81 -> 11.7 mm, vias 2 -> 1
- net Net-(U12-LITE): track 2.28 -> 8.89 mm
- net /processor/QSPI_CS: track 37.8 -> 44.2 mm
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- added copper zone on In2.Cu, net +3V3
- added copper zone on In1.Cu, net GND
- added copper zone on B.Cu, net GNDISO2
- removed copper zone on In1.Cu, net +3V3
- removed copper zone on In2.Cu, net GND
Other:
- board text added: "0"
- board text added: "1"
- board text added: "1s-4s"
- board text added: "2"
- board text added: "3"
- board text added: "4"
- board text added: "5"
- board text added: "6"
- board text added: "7"
- board text added: "Ain"
- board text added: "CAN"
- board text added: "High"
- board text added: "I2C0"
- board text added: "I2C1"
- board text added: "Low"
- board text added: "SWD"
- board text added: "UART"
- board text added: "boot"
- board text added: "rst"

Commit message: stuffs
Parts:
- added D13: LED, 1_Semi_Discrete_Diodes_SMD:D_0603, F.Cu at (116.9, 112.5)
- added D14: LED, 1_Semi_Discrete_Diodes_SMD:D_0603, F.Cu at (106.2, 112.4)
- added D7: LED, 1_Semi_Discrete_Diodes_SMD:D_0603, F.Cu at (141.9, 82.2)
- added R89: 300, 2_Passives_Resistors_SMD_IPC:R_1608_603_B, F.Cu at (142.9, 80.8)
- added R90: 300, 2_Passives_Resistors_SMD_IPC:R_1608_603_B, F.Cu at (117.0, 111.0)
- added R91: 300, 2_Passives_Resistors_SMD_IPC:R_1608_603_B, F.Cu at (105.5, 110.0)
- TP10, TP4: footprint 0_misc:test_point_0.8mm_square -> 0_misc:plated_hole_1.1x1.5mm
- moved TP4 6.26 mm to (165.4, 76.4)
- moved TP10 5.33 mm to (163.3, 76.4)
- moved C30 2.63 mm to (150.5, 78.1), turned to -90 degrees
- moved D10 2.12 mm to (165.8, 78.8), turned to -90 degrees
- moved R29 1.92 mm to (163.6, 79.1), turned to 180 degrees
- moved C2 1.43 mm to (111.8, 95.5)
- moved J4 0.28 mm to (158.7, 77.8)
Routing:
- net SWITCHING_3V3: track 144.8 -> 150.8 mm, vias 12 -> 13
- net EMG_LOW: track 71.1 -> 76.0 mm, vias 3 -> 2
- net EMG_HIGH: track 71.8 -> 74.7 mm, vias 3 -> 2
- net +5V: track 10.7 -> 12.7 mm
- net GNDREF: track 187.2 -> 189.2 mm, vias 9 -> 10
- net Net-(D7-A): track 0.00 -> 1.81 mm
- net Net-(D14-A): track 0.00 -> 1.58 mm
- net Net-(D13-A): track 0.00 -> 1.32 mm
- net Net-(SW4-A): track 10.8 -> 12.0 mm
- net +3V3: track 85.6 -> 86.6 mm, vias 33 -> 34
- net CHAN_0B_OUT: track 23.1 -> 24.0 mm, vias 2 -> 3
- net Net-(U3-BYP): track 7.18 -> 6.38 mm
- net GND: track 87.9 -> 87.7 mm, vias 44 -> 46
Other:
- board text added: "3V"
- board text added: "3VS"
- board text added: "5V"
- board text added: "H"
- board text added: "L"
- board text added: "SB 2023"

Commit message: stuffs
Parts:
- J2: moved to B.Cu
- J8: moved to F.Cu
- moved R21 2.95 mm to (130.4, 116.6), turned to 0 degrees
- moved R10 2.95 mm to (127.5, 118.0), turned to 180 degrees
- moved R9 2.95 mm to (130.4, 118.0), turned to 0 degrees
- moved R12 2.93 mm to (127.5, 116.6), turned to 180 degrees
- turned J2 to 180 degrees
- turned J8 to 0 degrees
Connections:
- D14 pad 1: GND -> GNDISO2
Routing:
- net GNDISO2: track 16.3 -> 20.2 mm, vias 12 -> 10
- net /SCL1: track 50.3 -> 47.5 mm
- net /SDA0: track 26.1 -> 28.0 mm
- net CHAN_0B_OUT: track 24.0 -> 25.4 mm
- net GND: track 87.7 -> 86.6 mm, vias 46 -> 45
- net /SCL0: track 28.0 -> 27.3 mm
- net +3V3: track 86.6 -> 86.8 mm, vias 34 -> 33
- net /SDA1: vias 2 -> 3
