File: eOPRA_interface/peripherals.kicad_sch (KiCad schematic)
At the start: 17 parts, among them Q7 Q_NMOS_GSD, SW1 SW_Push, U15 M41T81, Y3 Crystal

Commit message: schematic v1.0 finished
Parts:
- removed Q7: Q_NMOS_GSD, 1_Semi_TO_SOT:SOT-323FL, symbol 1.semi.discrete:Q_NMOS_GSD
- removed R20, R21, R22, R23, R24: R, symbol 2.passive:R
- removed R51: 500, 2_Passives_Resistors_SMD_IPC:R_2012_805_B, symbol 2.passive:R
- removed SW1 (x2): SW_Push, symbol 3.electromechanical.switch:SW_Push
- removed U15: M41T81, symbol 1.semi.ic.sensor:M41T81
- removed Y3: Crystal, symbol 2.passive:Crystal
- added C10 (x2): 0.01u, 2_Passives_Capacitors_SMD_IPC:C_1608_603_B, symbol 2.passive:C
- added R16 (x2): 300, 2_Passives_Resistors_SMD_IPC:R_1608_603_B, symbol 2.passive:R
- added R27 (x5): 10k, 2_Passives_Resistors_SMD_IPC:R_1608_603_B, symbol 2.passive:R
- added R4: 500, 2_Passives_Resistors_SMD_IPC:R_1608_603_B, symbol 2.passive:R
- added SW1: SW_Push, project_footprints:TL3365AF180QG, symbol 3.electromechanical.switch:SW_Push
- added SW7: Rotary_Encoder_Switch, project_footprints:PEC11S-929K-S0015, symbol 2.passive:Rotary_Encoder_Switch
- added U4: DS3231MZ+, 1_Semi_Misc:SOIC-8_3.9x4.9mm_P1.27mm, symbol 1.semi.ic.sensor:DS3231MZ+
- JP1: footprint (none) -> 0_misc:SolderJumper-2_P1.3mm_Open_RoundedPad1.0x1.5mm
- Q7: PN 4,11 -> (none)
- R16: PN 1,10 -> (none)
- R49: PN 1,5 -> (none)
- SP1: footprint 3_Electromechanical_Audio:13-9mm_Buzzer -> project_footprints:BUZZER; PN 5,1 -> (none)
- U12: footprint (none) -> project_footprints:TFT_BOB
Connections:
- net +3V3: now also JP1.2, R16.1, R16.2, R27.1, R27.2, R27.2, R4.1, U4.2 (VCC)
- net GND: now also C10.2, C10.2, SW1.2, SW1.4, SW7.C, SW7.S2, U4.5 (GND), U4.6 (VBAT)
- net ~{TFT_RESET}: now also R4.2, SW1.1, SW1.3
- net at SP1.1 (+): now also R16.1, R16.2
- net at U12.1 (LITE): now also JP1.1
- net TFT_DC: now reaches U12.7 (D/C)
- new net: R27.1, R27.1, SW7.A
- new net: R27.2, R27.2, SW7.B
- new net ENC_BUTTON: R27.1, SW7.S1
- new net ROT_ENC_A: C10.1, R27.2
- new net ROT_ENC_B: C10.1, R27.1
- new net SCL1: U4.8 (SCL)
- new net SDA1: U4.7 (SDA)
- no-connect marks 1 -> 3
Other:
- note added: "RTC"
- note removed: "Buttons"
- moved on the sheet: Q7, R16, R49, SP1, U12

Commit message: Version updates
Other:
- company: (none) -> Massachusetts Institute of Technology / MIT Media Lab
- title: (none) -> eOPRA Switch / Stimulation Controller
Changed lines of the file:
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@@
 (kicad_sch (version 20230121) (generator eeschema)
   (paper "A4")
+  (title_block
+    (title "eOPRA Switch / Stimulation Controller")
+    (date "2023-08-01")
+    (rev "1.0")
+    (company "Massachusetts Institute of Technology / MIT Media Lab")
+  )
   (junction (at 202.565 67.945) (diameter 0) (color 0 0 0 0)
   )

Commit message: starting layout
Connections:
- net ROT_ENC_A renamed ROT_ENC_0
- net ROT_ENC_B renamed ROT_ENC_1
Changed lines of the file:
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@@
     (effects (font (size 1.27 1.27)) (justify right))
   )
-  (hierarchical_label "ROT_ENC_A" (shape output) (at 222.885 122.555 0) (fields_autoplaced)
+  (hierarchical_label "ROT_ENC_0" (shape output) (at 222.885 122.555 0) (fields_autoplaced)
     (effects (font (size 1.27 1.27)) (justify left))
   )
-  (hierarchical_label "ROT_ENC_B" (shape output) (at 193.675 122.555 180) (fields_autoplaced)
+  (hierarchical_label "ROT_ENC_1" (shape output) (at 193.675 122.555 180) (fields_autoplaced)
     (effects (font (size 1.27 1.27)) (justify right))
   )

Commit message: before 4 layer
Connections:
- net GNDD is gone; now on net GND: Q7.2 (S), R49.1
Changed lines of the file:
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@@
+    )
+  )
+  (symbol (lib_id "0.power-symbols:GND") (at 220.345 78.105 0) (unit 1)
+    (in_bom yes) (on_board yes) (dnp no) (fields_autoplaced)
+    (property "Reference" "#PWR03" (at 220.345 84.455 0)
+      (effects (font (size 1.27 1.27)) hide)
+    )
+    (property "Value" "GND" (at 220.345 82.2405 0)
+      (effects (font (size 1.27 1.27)))
+    )
+    (property "Footprint" "" (at 220.345 78.105 0)
+      (effects (font (size 1.27 1.27)) hide)
+    )
+    (property "Datasheet" "" (at 220.345 78.105 0)
+      (effects (font (size 1.27 1.27)) hide)
+    )
+    (pin "1")
+    (instances
+      (project "eOPRA_interface"
+        (path "/9f7a57db-2daa-452d-a1aa-74a4ad8115df/a184413b-e455-471d-9900-996aedf52280"
+          (reference "#PWR03") (unit 1)
+        )
+      )
     )
   )
@@
         )
       )
-    )
-  )
-  (symbol (lib_id "0.power-symbols:GNDD") (at 220.345 78.105 0) (unit 1)
-    (in_bom yes) (on_board yes) (dnp no) (fields_autoplaced)
-    (property "Reference" "#PWR0126" (at 220.345 84.455 0)
-      (effects (font (size 1.27 1.27)) hide)
-    )
-    (property "Value" "GNDD" (at 220.345 82.5484 0)
-      (effects (font (size 1.27 1.27)))
-    )
-    (property "Footprint" "" (at 220.345 78.105 0)
-      (effects (font (size 1.27 1.27)) hide)
-    )
-    (property "Datasheet" "" (at 220.345 78.105 0)
-      (effects (font (size 1.27 1.27)) hide)
-    )
-    (pin "1")
-    (instances
-      (project "1.0"
-        (path "/628082f8-0394-4f00-be88-5631e8394d3a/a52b1568-2a4e-406c-adb6-97b12d034f30"
-          (reference "#PWR0126") (unit 1)
-        )
-      )
-      (project "eOPRA_interface"
-        (path "/9f7a57db-2daa-452d-a1aa-74a4ad8115df/a184413b-e455-471d-9900-996aedf52280"
-          (reference "#PWR013") (unit 1)
-        )
-      )

Commit message: preliminary finish
Parts:
- added C10: 0.1u, 2_Passives_Capacitors_SMD_IPC:C_1608_603_B, symbol 2.passive:C
- added C80: 10u, 2_Passives_Capacitors_SMD_IPC:C_2012_805_B, symbol 2.passive:C
Connections:
- net +3V3: now also C10.2, C80.2
- net GND: now also C10.1, C80.1
Changed lines of the file:
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@@
+    (stroke (width 0) (type default))
+  )
+  (wire (pts (xy 97.79 59.69) (xy 97.79 64.77))
     (stroke (width 0) (type default))
   )
@@
     (stroke (width 0) (type default))
   )
+  (wire (pts (xy 103.505 86.36) (xy 103.505 90.17))
+    (stroke (width 0) (type default))
+  )
   (wire (pts (xy 118.11 109.855) (xy 118.11 112.395))
     (stroke (width 0) (type default))
@@
     (stroke (width 0) (type default))
   )
+  (wire (pts (xy 103.505 97.79) (xy 103.505 99.695))
+    (stroke (width 0) (type default))
+  )
   (wire (pts (xy 205.74 122.555) (xy 204.47 122.555))
     (stroke (width 0) (type default))
@@
   )
   (wire (pts (xy 246.38 120.015) (xy 243.84 120.015))
+    (stroke (width 0) (type default))
+  )
+  (wire (pts (xy 97.79 46.99) (xy 97.79 52.07))
     (stroke (width 0) (type default))
   )
@@
     )
   )
+  (symbol (lib_id "2.passive:C") (at 103.505 93.98 180) (unit 1)
+    (in_bom yes) (on_board yes) (dnp no)
+    (property "Reference" "C80" (at 111.76 94.615 0)
+      (effects (font (size 1.27 1.27)) (justify left))
+    )
+    (property "Value" "10u" (at 111.76 92.71 0)
+      (effects (font (size 1.27 1.27)) (justify left))
+    )
+    (property "Footprint" "2_Passives_Capacitors_SMD_IPC:C_2012_805_B" (at 102.5398 90.17 0)
+      (effects (font (size 1.27 1.27)) hide)
+    )
+    (property "Datasheet" "~" (at 103.505 93.98 0)
+      (effects (font (size 1.27 1.27)) hide)
+    )
+    (property "PN" "2,2" (at 103.505 93.98 0)
+      (effects (font (size 1.27 1.27)) hide)
+    )
+    (pin "1")
+    (pin "2")
+    (instances
+      (project "1.0"
+        (path "/628082f8-0394-4f00-be88-5631e8394d3a/6fab7c9f-ac4d-49b1-a7fd-4592113b9455"
+          (reference "C80") (unit 1)
+        )
+      )
+      (project "eOPRA_interface"
+        (path "/9f7a57db-2daa-452d-a1aa-74a4ad8115df"
+          (reference "C3") (unit 1)
+        )
+        (path "/9f7a57db-2daa-452d-a1aa-74a4ad8115df/16a508a1-14d6-439d-afb0-bad239c786d4"
+          (reference "C20") (unit 1)
+        )
+        (path "/9f7a57db-2daa-452d-a1aa-74a4ad8115df/a184413b-e455-471d-9900-996aedf52280"
+          (reference "C31") (unit 1)
+        )
+      )
+    )
+  )
   (symbol (lib_id "2.passive:R") (at 118.11 116.205 0) (unit 1)
     (in_bom yes) (on_board yes) (dnp no)
@@
     )
   )
+  (symbol (lib_id "0.power-symbols:GND") (at 103.505 99.695 0) (unit 1)
+    (in_bom yes) (on_board yes) (dnp no) (fields_autoplaced)
+    (property "Reference" "#PWR046" (at 103.505 106.045 0)
+      (effects (font (size 1.27 1.27)) hide)
+    )
+    (property "Value" "GND" (at 103.505 103.8305 0)
+      (effects (font (size 1.27 1.27)))
+    )
+    (property "Footprint" "" (at 103.505 99.695 0)
+      (effects (font (size 1.27 1.27)) hide)
+    )
+    (property "Datasheet" "" (at 103.505 99.695 0)
+      (effects (font (size 1.27 1.27)) hide)
+    )
+    (pin "1")
+    (instances
+      (project "eOPRA_interface"
+        (path "/9f7a57db-2daa-452d-a1aa-74a4ad8115df/16a508a1-14d6-439d-afb0-bad239c786d4"
+          (reference "#PWR046") (unit 1)
+        )
+        (path "/9f7a57db-2daa-452d-a1aa-74a4ad8115df/a184413b-e455-471d-9900-996aedf52280"
+          (reference "#PWR036") (unit 1)
+        )
+      )
+    )
+  )
   (symbol (lib_id "2.passive:Jumper") (at 67.31 95.885 90) (unit 1)
     (in_bom yes) (on_board yes) (dnp no)
@@
         (path "/9f7a57db-2daa-452d-a1aa-74a4ad8115df/a184413b-e455-471d-9900-996aedf52280"
           (reference "#PWR037") (unit 1)
+        )
+      )
+    )
+  )
+  (symbol (lib_id "0.power-symbols:GND") (at 97.79 64.77 0) (unit 1)
+    (in_bom yes) (on_board yes) (dnp no) (fields_autoplaced)
+    (property "Reference" "#PWR020" (at 97.79 71.12 0)
+      (effects (font (size 1.27 1.27)) hide)
+    )
+    (property "Value" "GND" (at 97.79 68.9055 0)
+      (effects (font (size 1.27 1.27)))
+    )
+    (property "Footprint" "" (at 97.79 64.77 0)
+      (effects (font (size 1.27 1.27)) hide)
+    )
+    (property "Datasheet" "" (at 97.79 64.77 0)
+      (effects (font (size 1.27 1.27)) hide)
+    )
+    (pin "1")
+    (instances
+      (project "eOPRA_interface"
+        (path "/9f7a57db-2daa-452d-a1aa-74a4ad8115df/d165d604-1acf-4179-9574-6e327e7130e7"
+          (reference "#PWR020") (unit 1)
+        )
+        (path "/9f7a57db-2daa-452d-a1aa-74a4ad8115df/a184413b-e455-471d-9900-996aedf52280"
+          (reference "#PWR062") (unit 1)
         )
       )
@@
     )
   )
+  (symbol (lib_id "0.power-symbols:+3.3V") (at 103.505 86.36 0) (unit 1)
+    (in_bom yes) (on_board yes) (dnp no) (fields_autoplaced)
+    (property "Reference" "#PWR033" (at 103.505 90.17 0)
+      (effects (font (size 1.27 1.27)) hide)
+    )
+    (property "Value" "+3.3V" (at 103.505 82.8581 0)
+      (effects (font (size 1.27 1.27)))
+    )
+    (property "Footprint" "" (at 103.505 86.36 0)
+      (effects (font (size 1.27 1.27)) hide)
+    )
+    (property "Datasheet" "" (at 103.505 86.36 0)
+      (effects (font (size 1.27 1.27)) hide)
+    )
+    (pin "1")
+    (instances
+      (project "eOPRA_interface"
+        (path "/9f7a57db-2daa-452d-a1aa-74a4ad8115df/a184413b-e455-471d-9900-996aedf52280"
+          (reference "#PWR033") (unit 1)
+        )
+      )
+    )
+  )
   (symbol (lib_id "0.power-symbols:+3.3V") (at 69.85 86.36 0) (unit 1)
     (in_bom yes) (on_board yes) (dnp no) (fields_autoplaced)
@@
         )
       )
+    )
+  )
+  (symbol (lib_id "2.passive:C") (at 97.79 55.88 180) (unit 1)
+    (in_bom yes) (on_board yes) (dnp no) (fields_autoplaced)
+    (property "Reference" "C10" (at 100.711 55.0453 0)
+      (effects (font (size 1.27 1.27)) (justify right))
+    )
+    (property "Value" "0.1u" (at 100.711 57.5822 0)
+      (effects (font (size 1.27 1.27)) (justify right))
+    )
+    (property "Footprint" "2_Passives_Capacitors_SMD_IPC:C_1608_603_B" (at 96.8248 52.07 0)
+      (effects (font (size 1.27 1.27)) hide)
+    )
+    (property "Datasheet" "~" (at 97.79 55.88 0)
+      (effects (font (size 1.27 1.27)) hide)
+    )
+    (property "PN" "" (at 97.79 55.88 0)
+      (effects (font (size 1.27 1.27)) hide)
+    )
+    (pin "1")
+    (pin "2")
+    (instances
+      (project "1.0"
+        (path "/628082f8-0394-4f00-be88-5631e8394d3a/94532174-4d89-478b-a3e8-1052be6253fa"
+          (reference "C10") (unit 1)
+        )
+      )
+      (project "eOPRA_interface"
+        (path "/9f7a57db-2daa-452d-a1aa-74a4ad8115df/d165d604-1acf-4179-9574-6e327e7130e7"
+          (reference "C18") (unit 1)
+        )
+        (path "/9f7a57db-2daa-452d-a1aa-74a4ad8115df/a184413b-e455-471d-9900-996aedf52280"
+          (reference "C32") (unit 1)
+        )
+      )
+    )
+  )
+  (symbol (lib_id "0.power-symbols:+3.3V") (at 97.79 46.99 0) (unit 1)
+    (in_bom yes) (on_board yes) (dnp no) (fields_autoplaced)
+    (property "Reference" "#PWR019" (at 97.79 50.8 0)
+      (effects (font (size 1.27 1.27)) hide)
+    )
+    (property "Value" "+3.3V" (at 97.79 43.4881 0)
+      (effects (font (size 1.27 1.27)))
+    )
+    (property "Footprint" "" (at 97.79 46.99 0)
+      (effects (font (size 1.27 1.27)) hide)
+    )
+    (property "Datasheet" "" (at 97.79 46.99 0)
+      (effects (font (size 1.27 1.27)) hide)
+    )
+    (pin "1")
+    (instances
+      (project "eOPRA_interface"
+        (path "/9f7a57db-2daa-452d-a1aa-74a4ad8115df/d165d604-1acf-4179-9574-6e327e7130e7"
+          (reference "#PWR019") (unit 1)
+        )
+        (path "/9f7a57db-2daa-452d-a1aa-74a4ad8115df/a184413b-e455-471d-9900-996aedf52280"
+          (reference "#PWR044") (unit 1)
+        )
+      )

Commit message: stuff
Parts:
- removed C10: 0.1u, 2_Passives_Capacitors_SMD_IPC:C_1608_603_B, symbol 2.passive:C
- removed JP1: Jumper, 0_misc:SolderJumper-2_P1.3mm_Open_RoundedPad1.0x1.5mm, symbol 2.passive:Jumper
- added C33, C80: 1uF, 2_Passives_Capacitors_SMD_IPC:C_1005_402_A, symbol 2.passive:C
- added JP2: ~, 0_misc:SolderJumper-2_P1.3mm_Bridged_RoundedPad1.0x1.5mm, symbol 2.passive:Jumper_NC_Small
- added R27: 10k, 2_Passives_Resistors_SMD_IPC:R_1608_603_B, symbol 2.passive:R
- C10: value 0.01u -> 0.1uF; footprint 2_Passives_Capacitors_SMD_IPC:C_1608_603_B -> 2_Passives_Capacitors_SMD_IPC:C_1005_402_A; PN (none) -> 2,1
- C80: value 10u -> 1uF; footprint 2_Passives_Capacitors_SMD_IPC:C_2012_805_B -> 2_Passives_Capacitors_SMD_IPC:C_1005_402_A
- Q7: PN (none) -> 10,1
- R16: PN (none) -> 1,5
- R27, R49: PN (none) -> 1,2
- R4: PN (none) -> 1,4
- SP1: PN (none) -> 5,2
- SW1: PN (none) -> 9,4
- SW7: PN (none) -> 9,6
- U12: PN (none) -> 5,3
- U4: PN (none) -> 4,2
Connections:
- net +3V3: now also C80.2, JP2.2
- net ENC_BUTTON: now also C33.2, R27.2; no longer R27.1, SW7.S1
- net GND: now also C33.1, C80.1
- net at U12.1 (LITE): now also JP2.1
- new net switch: R27.1, R27.1, SW7.S1
Other:
- moved on the sheet: C10, C80, Q7, R16, R27, R4, R49, SP1, SW1, SW7, U12, U4

Commit message: stuff
Parts:
- removed R4: 500, 2_Passives_Resistors_SMD_IPC:R_1608_603_B, symbol 2.passive:R
- added R17: 1k, 2_Passives_Resistors_SMD_IPC:R_1005_402_A, symbol 2.passive:R
- Q7: value Q_NMOS_GSD -> RU1J002YNTCL
- SW7: Field4 PEC11S-929K-S0015 -> (none)
Connections:
- net +3V3: now also R17.1
- net ~{TFT_RESET}: now also R17.2
Changed lines of the file:
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@@
+    )
+  )
+  (symbol (lib_id "2.passive:R") (at 114.3 119.38 0) (unit 1)
+    (in_bom yes) (on_board yes) (dnp no)
+    (property "Reference" "R17" (at 110.49 120.015 0)
+      (effects (font (size 1.27 1.27)))
+    )
+    (property "Value" "1k" (at 108.585 118.11 0)
+      (effects (font (size 1.27 1.27)) (justify left))
+    )
+    (property "Footprint" "2_Passives_Resistors_SMD_IPC:R_1005_402_A" (at 112.522 119.38 90)
+      (effects (font (size 1.27 1.27)) hide)
+    )
+    (property "Datasheet" "~" (at 114.3 119.38 0)
+      (effects (font (size 1.27 1.27)) hide)
+    )
+    (property "PN" "1,3" (at 114.3 119.38 0)
+      (effects (font (size 1.27 1.27)) hide)
+    )
+    (pin "1")
+    (pin "2")
+    (instances
+      (project "eOPRA_interface"
+        (path "/9f7a57db-2daa-452d-a1aa-74a4ad8115df/d165d604-1acf-4179-9574-6e327e7130e7"
+          (reference "R17") (unit 1)
+        )
+        (path "/9f7a57db-2daa-452d-a1aa-74a4ad8115df/a184413b-e455-471d-9900-996aedf52280"
+          (reference "R18") (unit 1)
+        )
+      )
     )
   )
@@
       (effects (font (size 1.27 1.27)) (justify left))
     )
-    (property "Value" "Q_NMOS_GSD" (at 211.6074 72.8222 0)
+    (property "Value" "RU1J002YNTCL" (at 211.6074 72.8222 0)
       (effects (font (size 1.27 1.27)) (justify left))
     )
@@
     )
   )
-  (symbol (lib_id "2.passive:R") (at 114.3 119.38 0) (unit 1)
-    (in_bom yes) (on_board yes) (dnp no)
-    (property "Reference" "R4" (at 110.7755 120.9675 0)
-      (effects (font (size 1.27 1.27)))
-    )
-    (property "Value" "500" (at 110.7755 119.0465 0)
-      (effects (font (size 1.27 1.27)))
-    )
-    (property "Footprint" "2_Passives_Resistors_SMD_IPC:R_1608_603_B" (at 112.522 119.38 90)
-      (effects (font (size 1.27 1.27)) hide)
-    )
-    (property "Datasheet" "~" (at 114.3 119.38 0)
-      (effects (font (size 1.27 1.27)) hide)
-    )
-    (property "PN" "1,4" (at 114.3 119.38 0)
-      (effects (font (size 1.27 1.27)) hide)
-    )
-    (pin "1")
-    (pin "2")
-    (instances
-      (project "eOPRA_interface"
-        (path "/9f7a57db-2daa-452d-a1aa-74a4ad8115df/d165d604-1acf-4179-9574-6e327e7130e7"
-          (reference "R4") (unit 1)
-        )
-        (path "/9f7a57db-2daa-452d-a1aa-74a4ad8115df/a184413b-e455-471d-9900-996aedf52280"
-          (reference "R18") (unit 1)
-        )
-      )
-    )
-  )
   (symbol (lib_id "2.passive:C") (at 184.15 130.175 0) (unit 1)
     (in_bom yes) (on_board yes) (dnp no)
@@
       (effects (font (size 1.27 1.27)) hide)
     )
-    (property "Field4" "PEC11S-929K-S0015" (at 196.85 142.875 90)
-      (effects (font (size 1.27 1.27)) hide)
-    )
